File: PinCheck-4/fail_logic.kicad_sch (KiCad schematic)
At the start: 6 parts, among them U6 7408, U8 7432

Commit message: Daily sync 2025-08-27 16:57
Parts:
- removed D11: LED, symbol Device:LED
- removed R15: 1k, symbol Device:R
- C15: renamed from C9; footprint (none) -> Capacitor_SMD:C_0805_2012Metric
- C16: renamed from C11; footprint (none) -> Capacitor_SMD:C_0805_2012Metric
- U10: renamed from U6; footprint (none) -> Package_SO:SOIC-14_3.9x8.7mm_P1.27mm
- U11: renamed from U8; footprint (none) -> Package_SO:SOIC-14_3.9x8.7mm_P1.27mm
Connections:
- net R: now reaches U11.8
