File: PinCheck-4/pass_logic.kicad_sch (KiCad schematic)
At the start: 6 parts, among them U5 7408, U7 7432

Commit message: Daily sync 2025-08-27 16:57
Parts:
- removed D10: LED, symbol Device:LED
- removed R16: 1k, symbol Device:R
- C13: renamed from C10; footprint (none) -> Capacitor_SMD:C_0805_2012Metric
- C14: renamed from C7; footprint (none) -> Capacitor_SMD:C_0805_2012Metric
- U8: renamed from U5; footprint (none) -> Package_SO:SOIC-14_3.9x8.7mm_P1.27mm
- U9: renamed from U7; footprint (none) -> Package_SO:SOIC-14_3.9x8.7mm_P1.27mm
Connections:
- net G: now reaches U9.8
