File: PinCheck-4/pass_fail_logic.kicad_sch (KiCad schematic)
At the start: 6 parts, among them U10 4072, U8 7408, U9 7408

Commit message: Daily sync 2025-08-28 16:55
Connections:
- net G0: no longer names the net of U10.2, U8.3
- net G1: no longer names the net of U10.3, U8.6
- net G2: no longer names the net of U10.4, U8.8
- net G3: no longer names the net of U10.5, U8.11
- net R0: no longer names the net of U10.9, U9.3
- net R1: no longer names the net of U10.10, U9.6
- net R2: no longer names the net of U10.11, U9.8
- net R3: no longer names the net of U10.12, U9.11
- no-connect marks 1 -> 0
Other:
- moved on the sheet: C13, C14, C15, U10A, U10B, U10C, U8A, U8B, U8C, U8D, U9A, U9B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

Commit message: Daily sync 2025-08-29 22:48
Parts:
- C13, C14, C15: Manufacturer Part No (none) -> 0805B104K160CT
- U10: Manufacturer Part No (none) -> CD4072BM96
- U8, U9: Manufacturer Part No (none) -> 74HC08D
Changed lines of the file:
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@@
 			)
 		)
-		(property "Description" ""
+		(property "Description" "AND Gate IC 4 Channel 14-SOIC"
+			(at 48.26 130.81 0)
+			(effects
+				(font
+					(size 1.27 1.27)
+				)
+				(hide yes)
+			)
+		)
+		(property "Manufacturer Part No" "74HC08D"
 			(at 48.26 130.81 0)
 			(effects
@@
 			)
 		)
-		(property "Description" ""
+		(property "Description" "AND Gate IC 4 Channel 14-SOIC"
+			(at 171.45 130.81 0)
+			(effects
+				(font
+					(size 1.27 1.27)
+				)
+				(hide yes)
+			)
+		)
+		(property "Manufacturer Part No" "74HC08D"
 			(at 171.45 130.81 0)
 			(effects
@@
 			)
 		)
-		(property "Description" ""
+		(property "Description" "AND Gate IC 4 Channel 14-SOIC"
+			(at 88.9 130.81 0)
+			(effects
+				(font
+					(size 1.27 1.27)
+				)
+				(hide yes)
+			)
+		)
+		(property "Manufacturer Part No" "74HC08D"
 			(at 88.9 130.81 0)
 			(effects
@@
 			)
 		)
-		(property "Description" ""
+		(property "Description" "AND Gate IC 4 Channel 14-SOIC"
+			(at 48.26 60.96 0)
+			(effects
+				(font
+					(size 1.27 1.27)
+				)
+				(hide yes)
+			)
+		)
+		(property "Manufacturer Part No" "74HC08D"
 			(at 48.26 60.96 0)
 			(effects
@@
 			)
 		)
-		(property "Description" "Dual 4 input OR gate"
+		(property "Description" "OR Gate IC 2 Channel 14-SOIC"
+			(at 204.47 33.02 0)
+			(effects
+				(font
+					(size 1.27 1.27)
+				)
+				(hide yes)
+			)
+		)
+		(property "Manufacturer Part No" "CD4072BM96"
 			(at 204.47 33.02 0)
 			(effects
@@
 			)
 		)
-		(property "Description" "Unpolarized capacitor"
+		(property "Description" "SMD Multilayer Ceramic Capacitor, 0.1 µF, 16 V, 0805 [2012 Metric], ± 10%, X7R"
+			(at 245.11 110.49 0)
+			(effects
+				(font
+					(size 1.27 1.27)
+				)
+				(hide yes)
+			)
+		)
+		(property "Manufacturer Part No" "0805B104K160CT"
 			(at 245.11 110.49 0)
 			(effects
@@
 			)
 		)
-		(property "Description" "Dual 4 input OR gate"
+		(property "Description" "OR Gate IC 2 Channel 14-SOIC"
+			(at 260.35 129.54 0)
+			(effects
+				(font
+					(size 1.27 1.27)
+				)
+				(hide yes)
+			)
+		)
+		(property "Manufacturer Part No" "CD4072BM96"
 			(at 260.35 129.54 0)
 			(effects
@@
 			)
 		)
-		(property "Description" ""
+		(property "Description" "AND Gate IC 4 Channel 14-SOIC"
+			(at 129.54 60.96 0)
+			(effects
+				(font
+					(size 1.27 1.27)
+				)
+				(hide yes)
+			)
+		)
+		(property "Manufacturer Part No" "74HC08D"
 			(at 129.54 60.96 0)
 			(effects
@@
 			)
 		)
-		(property "Description" ""
+		(property "Description" "AND Gate IC 4 Channel 14-SOIC"
+			(at 171.45 60.96 0)
+			(effects
+				(font
+					(size 1.27 1.27)
+				)
+				(hide yes)
+			)
+		)
+		(property "Manufacturer Part No" "74HC08D"
 			(at 171.45 60.96 0)
 			(effects
@@
 			)
 		)
-		(property "Description" ""
+		(property "Description" "AND Gate IC 4 Channel 14-SOIC"
+			(at 88.9 60.96 0)
+			(effects
+				(font
+					(size 1.27 1.27)
+				)
+				(hide yes)
+			)
+		)
+		(property "Manufacturer Part No" "74HC08D"
 			(at 88.9 60.96 0)
 			(effects
@@
 			)
 		)
-		(property "Description" "Unpolarized capacitor"
+		(property "Description" "SMD Multilayer Ceramic Capacitor, 0.1 µF, 16 V, 0805 [2012 Metric], ± 10%, X7R"
+			(at 33.02 40.64 0)
+			(effects
+				(font
+					(size 1.27 1.27)
+				)
+				(hide yes)
+			)
+		)
+		(property "Manufacturer Part No" "0805B104K160CT"
 			(at 33.02 40.64 0)
 			(effects
@@
 			)
 		)
-		(property "Description" "Dual 4 input OR gate"
+		(property "Description" "OR Gate IC 2 Channel 14-SOIC"
+			(at 204.47 102.87 0)
+			(effects
+				(font
+					(size 1.27 1.27)
+				)
+				(hide yes)
+			)
+		)
+		(property "Manufacturer Part No" "CD4072BM96"
 			(at 204.47 102.87 0)
 			(effects
@@
 			)
 		)
-		(property "Description" ""
+		(property "Description" "AND Gate IC 4 Channel 14-SOIC"
+			(at 129.54 130.81 0)
+			(effects
+				(font
+					(size 1.27 1.27)
+				)
+				(hide yes)
+			)
+		)
+		(property "Manufacturer Part No" "74HC08D"
 			(at 129.54 130.81 0)
 			(effects
@@
 			)
 		)
-		(property "Description" "Unpolarized capacitor"
+		(property "Description" "SMD Multilayer Ceramic Capacitor, 0.1 µF, 16 V, 0805 [2012 Metric], ± 10%, X7R"
 			(at 33.02 110.49 0)
 			(effects
+				(font
+					(size 1.27 1.27)
+				)
+				(hide yes)
+			)
+		)
+		(property "Manufacturer Part No" "0805B104K160CT"
+			(at 33.02 110.49 0)
+			(effects

Commit message: Daily sync 2025-08-30 13:49
Parts:
- renumbered U9 to U10, U10 to U11, U8 to U9
Changed lines of the file:
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@@
 		(dnp no)
 		(fields_autoplaced yes)
-		(property "Reference" "U9"
+		(property "Reference" "U10"
 			(at 58.42 124.3898 0)
 			(effects
@@
 			(project "PinCheck-4"
 				(path "/8e21fa9a-50eb-4ff7-ab75-73c4d6c5f942/18f07d9e-ab3c-42ec-9938-33f6c3daee65"
-					(reference "U9")
+					(reference "U10")
 					(unit 1)
 				)
@@
 		(dnp no)
 		(fields_autoplaced yes)
-		(property "Reference" "U9"
+		(property "Reference" "U10"
 			(at 181.61 124.3898 0)
 			(effects
@@
 			(project "PinCheck-4"
 				(path "/8e21fa9a-50eb-4ff7-ab75-73c4d6c5f942/18f07d9e-ab3c-42ec-9938-33f6c3daee65"
-					(reference "U9")
+					(reference "U10")
 					(unit 4)
 				)
@@
 		(dnp no)
 		(fields_autoplaced yes)
-		(property "Reference" "U9"
+		(property "Reference" "U10"
 			(at 99.06 124.3898 0)
 			(effects
@@
 			(project "PinCheck-4"
 				(path "/8e21fa9a-50eb-4ff7-ab75-73c4d6c5f942/18f07d9e-ab3c-42ec-9938-33f6c3daee65"
-					(reference "U9")
+					(reference "U10")
 					(unit 2)
 				)
@@
 		(dnp no)
 		(fields_autoplaced yes)
-		(property "Reference" "U8"
+		(property "Reference" "U9"
 			(at 58.42 54.5398 0)
 			(effects
@@
 			(project "PinCheck-4"
 				(path "/8e21fa9a-50eb-4ff7-ab75-73c4d6c5f942/18f07d9e-ab3c-42ec-9938-33f6c3daee65"
-					(reference "U8")
+					(reference "U9")
 					(unit 1)
 				)
@@
 		(dnp no)
 		(fields_autoplaced yes)
-		(property "Reference" "#PWR043"
+		(property "Reference" "#PWR047"
 			(at 33.02 123.19 0)
 			(effects
@@
 			(project "PinCheck-4"
 				(path "/8e21fa9a-50eb-4ff7-ab75-73c4d6c5f942/18f07d9e-ab3c-42ec-9938-33f6c3daee65"
-					(reference "#PWR043")
+					(reference "#PWR047")
 					(unit 1)
 				)
@@
 		(dnp no)
 		(fields_autoplaced yes)
-		(property "Reference" "#PWR050"
+		(property "Reference" "#PWR054"
 			(at 260.35 151.13 0)
 			(effects
@@
 			(project "PinCheck-4"
 				(path "/8e21fa9a-50eb-4ff7-ab75-73c4d6c5f942/18f07d9e-ab3c-42ec-9938-33f6c3daee65"
-					(reference "#PWR050")
+					(reference "#PWR054")
 					(unit 1)
 				)
@@
 		(dnp no)
 		(fields_autoplaced yes)
-		(property "Reference" "U10"
+		(property "Reference" "U11"
 			(at 204.47 24.13 0)
 			(effects
@@
 			(project "PinCheck-4"
 				(path "/8e21fa9a-50eb-4ff7-ab75-73c4d6c5f942/18f07d9e-ab3c-42ec-9938-33f6c3daee65"
-					(reference "U10")
+					(reference "U11")
 					(unit 1)
 				)
@@
 		(dnp no)
 		(fields_autoplaced yes)
-		(property "Reference" "#PWR048"
+		(property "Reference" "#PWR052"
 			(at 245.11 123.19 0)
 			(effects
@@
 			(project "PinCheck-4"
 				(path "/8e21fa9a-50eb-4ff7-ab75-73c4d6c5f942/18f07d9e-ab3c-42ec-9938-33f6c3daee65"
-					(reference "#PWR048")
+					(reference "#PWR052")
 					(unit 1)
 				)
@@
 		(dnp no)
 		(fields_autoplaced yes)
-		(property "Reference" "U10"
+		(property "Reference" "U11"
 			(at 266.7 128.2699 0)
 			(effects
@@
 			(project "PinCheck-4"
 				(path "/8e21fa9a-50eb-4ff7-ab75-73c4d6c5f942/18f07d9e-ab3c-42ec-9938-33f6c3daee65"
-					(reference "U10")
+					(reference "U11")
 					(unit 3)
 				)
@@
 		(dnp no)
 		(fields_autoplaced yes)
-		(property "Reference" "U8"
+		(property "Reference" "U9"
 			(at 139.7 54.5398 0)
 			(effects
@@
 			(project "PinCheck-4"
 				(path "/8e21fa9a-50eb-4ff7-ab75-73c4d6c5f942/18f07d9e-ab3c-42ec-9938-33f6c3daee65"
-					(reference "U8")
+					(reference "U9")
 					(unit 3)
 				)
@@
 		(dnp no)
 		(fields_autoplaced yes)
-		(property "Reference" "#PWR046"
+		(property "Reference" "#PWR050"
 			(at 171.45 85.09 0)
 			(effects
@@
 			(project "PinCheck-4"
 				(path "/8e21fa9a-50eb-4ff7-ab75-73c4d6c5f942/18f07d9e-ab3c-42ec-9938-33f6c3daee65"
-					(reference "#PWR046")
+					(reference "#PWR050")
 					(unit 1)
 				)
@@
 		(dnp no)
 		(fields_autoplaced yes)
-		(property "Reference" "U8"
+		(property "Reference" "U9"
 			(at 181.61 54.5398 0)
 			(effects
@@
 			(project "PinCheck-4"
 				(path "/8e21fa9a-50eb-4ff7-ab75-73c4d6c5f942/18f07d9e-ab3c-42ec-9938-33f6c3daee65"
-					(reference "U8")
+					(reference "U9")
 					(unit 4)
 				)
@@
 		(dnp no)
 		(fields_autoplaced yes)
-		(property "Reference" "#PWR045"
+		(property "Reference" "#PWR049"
 			(at 48.26 104.14 0)
 			(effects
@@
 			(project "PinCheck-4"
 				(path "/8e21fa9a-50eb-4ff7-ab75-73c4d6c5f942/18f07d9e-ab3c-42ec-9938-33f6c3daee65"
-					(reference "#PWR045")
+					(reference "#PWR049")
 					(unit 1)
 				)
@@
 		(dnp no)
 		(fields_autoplaced yes)
-		(property "Reference" "#PWR049"
+		(property "Reference" "#PWR053"
 			(at 260.35 104.14 0)
 			(effects
@@
 			(project "PinCheck-4"
 				(path "/8e21fa9a-50eb-4ff7-ab75-73c4d6c5f942/18f07d9e-ab3c-42ec-9938-33f6c3daee65"
-					(reference "#PWR049")
+					(reference "#PWR053")
 					(unit 1)
 				)
@@
 		(dnp no)
 		(fields_autoplaced yes)
-		(property "Reference" "U8"
+		(property "Reference" "U9"
 			(at 99.06 54.5398 0)
 			(effects
@@
 			(project "PinCheck-4"
 				(path "/8e21fa9a-50eb-4ff7-ab75-73c4d6c5f942/18f07d9e-ab3c-42ec-9938-33f6c3daee65"
-					(reference "U8")
+					(reference "U9")
 					(unit 2)
 				)
@@
 		(dnp no)
 		(fields_autoplaced yes)
-		(property "Reference" "#PWR042"
+		(property "Reference" "#PWR046"
 			(at 33.02 53.34 0)
 			(effects
@@
 			(project "PinCheck-4"
 				(path "/8e21fa9a-50eb-4ff7-ab75-73c4d6c5f942/18f07d9e-ab3c-42ec-9938-33f6c3daee65"
-					(reference "#PWR042")
+					(reference "#PWR046")
 					(unit 1)
 				)
@@
 		(dnp no)
 		(fields_autoplaced yes)
-		(property "Reference" "U10"
+		(property "Reference" "U11"
 			(at 204.47 93.98 0)
 			(effects
@@
 			(project "PinCheck-4"
 				(path "/8e21fa9a-50eb-4ff7-ab75-73c4d6c5f942/18f07d9e-ab3c-42ec-9938-33f6c3daee65"
-					(reference "U10")
+					(reference "U11")
 					(unit 2)
 				)
@@
 		(dnp no)
 		(fields_autoplaced yes)
-		(property "Reference" "#FLG03"
+		(property "Reference" "#FLG04"
 			(at 174.625 146.05 0)
 			(effects
@@
 			(project ""
 				(path "/8e21fa9a-50eb-4ff7-ab75-73c4d6c5f942/18f07d9e-ab3c-42ec-9938-33f6c3daee65"
-					(reference "#FLG03")
+					(reference "#FLG04")
 					(unit 1)
 				)
@@
 		(dnp no)
 		(fields_autoplaced yes)
-		(property "Reference" "U9"
+		(property "Reference" "U10"
 			(at 139.7 124.3898 0)
 			(effects
@@
 			(project "PinCheck-4"
 				(path "/8e21fa9a-50eb-4ff7-ab75-73c4d6c5f942/18f07d9e-ab3c-42ec-9938-33f6c3daee65"
-					(reference "U9")
+					(reference "U10")
 					(unit 3)
 				)
@@
 		(dnp no)
 		(fields_autoplaced yes)
-		(property "Reference" "#PWR047"
+		(property "Reference" "#PWR051"
 			(at 171.45 154.94 0)
 			(effects
@@
 			(project "PinCheck-4"
 				(path "/8e21fa9a-50eb-4ff7-ab75-73c4d6c5f942/18f07d9e-ab3c-42ec-9938-33f6c3daee65"
-					(reference "#PWR047")
+					(reference "#PWR051")
 					(unit 1)
 				)
@@
 		(dnp no)
 		(fields_autoplaced yes)
-		(property "Reference" "#PWR044"
+		(property "Reference" "#PWR048"
 			(at 48.26 34.29 0)
 			(effects
@@
 			(project "PinCheck-4"
 				(path "/8e21fa9a-50eb-4ff7-ab75-73c4d6c5f942/18f07d9e-ab3c-42ec-9938-33f6c3daee65"
-					(reference "#PWR044")
+					(reference "#PWR048")
 					(unit 1)
 				)
