File: PinCheck-4/PinCheck-4.kicad_sch (KiCad schematic)
At the start: 40 parts, among them J1 DB9 In, J2 LEMHAL Header, U10 NE555D, U2 4017, U3 74HC14, U4 7408, U5 7408, U6 7408, U7 7432, U8 7432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

Commit message: Daily sync 2025-08-27 12:04
Parts:
- removed C1, C2, C3, C6, C7, C8, C9: 100n, symbol Device:C
- removed C4: 10n, symbol Device:C
- removed C5: 4.7u, symbol Device:C
- removed D1, D2, D3, D4, D5: LED, symbol Device:LED
- removed J1: DB9 In, symbol Connector:Conn_01x04_Socket
- removed J2: LEMHAL Header, symbol Connector:Conn_01x04_Socket
- removed R1, R10, R3, R4, R5, R6, R7, R8, R9: 1k, symbol Device:R
- removed R11, R12, R13, R14: 100k, symbol Device:R
- removed R2: 10k, symbol Device:R
- removed RV1: 100k, symbol Device:R_Potentiometer
- removed U10: NE555D, Package_SO:SOIC-8_3.9x4.9mm_P1.27mm, symbol Timer:NE555D
- removed U2: 4017, symbol 4xxx:4017
- removed U3: 74HC14, symbol 74xx:74HC14
- removed U4, U5, U6: 7408, symbol 74xx_IEEE:7408
- removed U7, U8, U9: 7432, symbol 74xx_IEEE:7432
Connections:
- no-connect marks 2 -> 0
Other:
- added sheet Clock_Logic (clock_logic.kicad_sch)
- added sheet Fail_Logic (fail_logic.kicad_sch)
- added sheet Pass_Logic (pass_logic.kicad_sch)
- added sheet Seq_Logic (seq_logic.kicad_sch)
- note removed: "ADD ESD array"
- note removed: "ADD a selector to change DB9 as per mode TOP / BOTTOM (IGBT & OVP)"
- company: (none) -> Igor Oliveira
- title: (none) -> PinCheck - 4 Pin Cable (LEMHAL)

Commit message: Daily sync 2025-08-27 16:57
Parts:
- added C1, C2, C3: 10u, Capacitor_SMD:C_0805_2012Metric, symbol Device:C
- added D1, D2, D3, D4, D5, D6: LED, LED_THT:LED_D3.0mm_Clear, symbol Device:LED
- added D7: LED_Dual_AAK, LED_THT:LED_D3.0mm-3, symbol Device:LED_Dual_AAK
- added R1, R3, R4, R5, R6, R8: 2.2k, Resistor_SMD:R_0805_2012Metric, symbol Device:R
- added R2, R7: 2.7k, Resistor_SMD:R_0805_2012Metric, symbol Device:R
Connections:
- new net: D1.1 (K), R1.1
- new net: D6.1 (K), R6.1
- new net: D5.1 (K), R5.1
- new net: D4.1 (K), R4.1
- new net: D7.1 (A1), R7.1
- new net: D7.2 (A2), R8.1
- new net: D3.1 (K), R3.1
- new net: D2.1 (K), R2.1
- new net CLK: D2.2 (A)
- new net G: R8.2
- new net GND: C1.2, C2.2, C3.2, D7.3 (K), R1.2, R2.2, R3.2, R4.2, R5.2, R6.2
- new net Q0: D3.2 (A)
- new net Q1: D4.2 (A)
- new net Q2: D5.2 (A)
- new net Q3: D6.2 (A)
- new net R: R7.2
- new net VCC: C1.1, C2.1, C3.1, D1.2 (A)
Other:
- added sheet SwitchLogic (spdt_logic.kicad_sch)
- note added: "EXTRA DECOUPLING"
- note added: "STATUS"

Commit message: Daily sync 2025-08-27 22:21
Other:
- sheet Pass_Logic renamed Pass_Fail_Logic
- removed sheet Fail_Logic
- sheet Pass_Fail_Logic: file pass_logic.kicad_sch -> pass_fail_logic.kicad_sch
Changed lines of the file:
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@@
 			(color 0 0 0 0.0000)
 		)
-		(property "Sheetname" "Pass_Logic"
+		(property "Sheetname" "Pass_Fail_Logic"
 			(at 153.67 91.9984 0)
 			(effects
@@
 			)
 		)
-		(property "Sheetfile" "pass_logic.kicad_sch"
+		(property "Sheetfile" "pass_fail_logic.kicad_sch"
 			(at 153.67 123.7746 0)
 			(effects
@@
 				)
 			)
-		)
-	)
-	(sheet
-		(at 181.61 53.34)
-		(size 54.61 30.48)
-		(exclude_from_sim no)
-		(in_bom yes)
-		(on_board yes)
-		(dnp no)
-		(fields_autoplaced yes)
-		(stroke
-			(width 0.1524)
-			(type solid)
-		)
-		(fill
-			(color 0 0 0 0.0000)
-		)
-		(property "Sheetname" "Fail_Logic"
-			(at 181.61 52.6284 0)
-			(effects
-				(font
-					(size 1.27 1.27)
-				)
-				(justify left bottom)
-			)
-		)
-		(property "Sheetfile" "fail_logic.kicad_sch"
-			(at 181.61 84.4046 0)
-			(effects
-				(font
-					(size 1.27 1.27)
-				)
-				(justify left top)
-			)
-		)
-		(instances
-			(project "PinCheck-4"
-				(path "/8e21fa9a-50eb-4ff7-ab75-73c4d6c5f942"
-					(page "6")
-				)
-			)

Commit message: Daily sync 2025-08-29 22:48
Parts:
- D1, D3, D4, D5, D6: Manufacturer Part No (none) -> L-934GD
- D2: value LED -> Y LED; Manufacturer Part No (none) -> L-934ND
- D7: Manufacturer Part No (none) -> L-93WEGW
- R1, R3, R4, R5, R6, R8: Manufacturer Part No (none) -> MC01W080512K2
- R2, R7: Manufacturer Part No (none) -> MCMR08X2701FTL
Changed lines of the file:
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@@
 			)
 		)
-		(property "Description" "Light emitting diode"
+		(property "Description" "LED, Low Power, Green, Through Hole, T-1 (3mm), 20 mA, 2.2 V, 568 nm"
 			(at 21.59 168.91 0)
 			(effects
@@
 			)
 		)
+		(property "Manufacturer Part No" "L-934GD"
+			(at 21.59 168.91 90)
+			(effects
+				(font
+					(size 1.27 1.27)
+				)
+				(hide yes)
+			)
+		)
 		(pin "1"
 		)
@@
 			)
 		)
+		(property "Manufacturer Part No" ""
+			(at 124.46 179.07 0)
+			(effects
+				(font
+					(size 1.27 1.27)
+				)
+				(hide yes)
+			)
+		)
 		(pin "1"
 		)
@@
 			)
 		)
-		(property "Description" "Resistor"
+		(property "Description" "SMD Chip Resistor, 2.2 kohm, ± 1%, 100 mW, 0805 [2012 Metric], Thick Film, General Purpose"
+			(at 21.59 179.07 0)
+			(effects
+				(font
+					(size 1.27 1.27)
+				)
+				(hide yes)
+			)
+		)
+		(property "Manufacturer Part No" "MC01W080512K2"
 			(at 21.59 179.07 0)
 			(effects
@@
 			)
 		)
-		(property "Description" "Light emitting diode"
+		(property "Description" "LED, Low Power, Green, Through Hole, T-1 (3mm), 20 mA, 2.2 V, 568 nm"
 			(at 72.39 168.91 0)
 			(effects
@@
 			)
 		)
+		(property "Manufacturer Part No" "L-934GD"
+			(at 72.39 168.91 90)
+			(effects
+				(font
+					(size 1.27 1.27)
+				)
+				(hide yes)
+			)
+		)
 		(pin "1"
 		)
@@
 			)
 		)
-		(property "Description" "Light emitting diode"
+		(property "Description" "LED, Low Power, Green, Through Hole, T-1 (3mm), 20 mA, 2.2 V, 568 nm"
 			(at 62.23 168.91 0)
 			(effects
@@
 			)
 		)
+		(property "Manufacturer Part No" "L-934GD"
+			(at 62.23 168.91 90)
+			(effects
+				(font
+					(size 1.27 1.27)
+				)
+				(hide yes)
+			)
+		)
 		(pin "1"
 		)
@@
 			)
 		)
-		(property "Description" "Resistor"
+		(property "Description" "SMD Chip Resistor, 2.2 kohm, ± 1%, 100 mW, 0805 [2012 Metric], Thick Film, General Purpose"
+			(at 52.07 179.07 0)
+			(effects
+				(font
+					(size 1.27 1.27)
+				)
+				(hide yes)
+			)
+		)
+		(property "Manufacturer Part No" "MC01W080512K2"
 			(at 52.07 179.07 0)
 			(effects
@@
 			)
 		)
-		(property "Description" "Dual LED, common cathode on pin 3"
+		(property "Description" "LED, Green, Red, Through Hole, T-1 (3mm), 60 °, Round, R 30mA, G 25mA"
 			(at 90.17 177.8 0)
+			(effects
+				(font
+					(size 1.27 1.27)
+				)
+				(hide yes)
+			)
+		)
+		(property "Manufacturer Part No" "L-93WEGW"
+			(at 90.17 177.8 90)
 			(effects
 				(font
@@
 			)
 		)
-		(property "Description" "Resistor"
+		(property "Description" "SMD Chip Resistor, 2.2 kohm, ± 1%, 100 mW, 0805 [2012 Metric], Thick Film, General Purpose"
+			(at 41.91 179.07 0)
+			(effects
+				(font
+					(size 1.27 1.27)
+				)
+				(hide yes)
+			)
+		)
+		(property "Manufacturer Part No" "MC01W080512K2"
 			(at 41.91 179.07 0)
 			(effects
@@
 			)
 		)
-		(property "Description" "Resistor"
+		(property "Description" "SMD Chip Resistor, 2.2 kohm, ± 1%, 100 mW, 0805 [2012 Metric], Thick Film, General Purpose"
+			(at 92.71 166.37 0)
+			(effects
+				(font
+					(size 1.27 1.27)
+				)
+				(hide yes)
+			)
+		)
+		(property "Manufacturer Part No" "MC01W080512K2"
 			(at 92.71 166.37 0)
 			(effects
@@
 			)
 		)
+		(property "Manufacturer Part No" ""
+			(at 147.32 179.07 0)
+			(effects
+				(font
+					(size 1.27 1.27)
+				)
+				(hide yes)
+			)
+		)
 		(pin "1"
 		)
@@
 			)
 		)
-		(property "Description" "Light emitting diode"
+		(property "Description" "LED, Low Power, Green, Through Hole, T-1 (3mm), 20 mA, 2.2 V, 568 nm"
 			(at 41.91 168.91 0)
 			(effects
@@
 			)
 		)
+		(property "Manufacturer Part No" "L-934GD"
+			(at 41.91 168.91 90)
+			(effects
+				(font
+					(size 1.27 1.27)
+				)
+				(hide yes)
+			)
+		)
 		(pin "1"
 		)
@@
 			)
 		)
-		(property "Value" "LED"
+		(property "Value" "Y LED"
 			(at 35.56 171.7674 90)
 			(effects
@@
 			)
 		)
-		(property "Description" "Light emitting diode"
+		(property "Description" "LED, Low Power, Orange, Through Hole, T-1 (3mm), 20 mA, 2.05 V, 610 nm"
 			(at 31.75 168.91 0)
 			(effects
@@
 			)
 		)
+		(property "Manufacturer Part No" "L-934ND"
+			(at 31.75 168.91 90)
+			(effects
+				(font
+					(size 1.27 1.27)
+				)
+				(hide yes)
+			)
+		)
 		(pin "1"
 		)
@@
 			)
 		)
-		(property "Description" "Resistor"
+		(property "Description" "SMD Chip Resistor, 2.2 kohm, ± 1%, 100 mW, 0805 [2012 Metric], Thick Film, General Purpose"
+			(at 62.23 179.07 0)
+			(effects
+				(font
+					(size 1.27 1.27)
+				)
+				(hide yes)
+			)
+		)
+		(property "Manufacturer Part No" "MC01W080512K2"
 			(at 62.23 179.07 0)
 			(effects
@@
 			)
 		)
+		(property "Manufacturer Part No" ""
+			(at 135.89 179.07 0)
+			(effects
+				(font
+					(size 1.27 1.27)
+				)
+				(hide yes)
+			)
+		)
 		(pin "1"
 		)
@@
 			)
 		)
-		(property "Description" "Resistor"
+		(property "Description" "SMD Chip Resistor, Ceramic, 2.7 kohm, ± 1%, 125 mW, 0805 [2012 Metric], Thick Film"
+			(at 31.75 179.07 0)
+			(effects
+				(font
+					(size 1.27 1.27)
+				)
+				(hide yes)
+			)
+		)
+		(property "Manufacturer Part No" "MCMR08X2701FTL"
 			(at 31.75 179.07 0)
 			(effects
@@
 			)
 		)
-		(property "Description" "Resistor"
+		(property "Description" "SMD Chip Resistor, Ceramic, 2.7 kohm, ± 1%, 125 mW, 0805 [2012 Metric], Thick Film"
+			(at 87.63 166.37 0)
+			(effects
+				(font
+					(size 1.27 1.27)
+				)
+				(hide yes)
+			)
+		)
+		(property "Manufacturer Part No" "MCMR08X2701FTL"
 			(at 87.63 166.37 0)
 			(effects
@@
 			)
 		)
-		(property "Description" "Light emitting diode"
+		(property "Description" "LED, Low Power, Green, Through Hole, T-1 (3mm), 20 mA, 2.2 V, 568 nm"
 			(at 52.07 168.91 0)
 			(effects
@@
 			)
 		)
+		(property "Manufacturer Part No" "L-934GD"
+			(at 52.07 168.91 90)
+			(effects
+				(font
+					(size 1.27 1.27)
+				)
+				(hide yes)
+			)
+		)
 		(pin "1"
 		)
@@
 			)
 		)
-		(property "Description" "Resistor"
+		(property "Description" "SMD Chip Resistor, 2.2 kohm, ± 1%, 100 mW, 0805 [2012 Metric], Thick Film, General Purpose"
 			(at 72.39 179.07 0)
 			(effects
+				(font
+					(size 1.27 1.27)
+				)
+				(hide yes)
+			)
+		)
+		(property "Manufacturer Part No" "MC01W080512K2"
+			(at 72.39 179.07 0)
+			(effects

Commit message: Daily sync 2025-08-30 13:49
Connections:
- net Q0 renamed S0
- net Q1 renamed S1
- net Q2 renamed S2
- net Q3 renamed S3
Changed lines of the file:
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@@
 		)
 	)
-	(global_label "Q0"
+	(global_label "S2"
 		(shape input)
-		(at 41.91 165.1 90)
+		(at 62.23 165.1 90)
 		(fields_autoplaced yes)
 		(effects
@@
 		)
 		(property "Intersheetrefs" "${INTERSHEET_REFS}"
-			(at 41.91 159.5748 90)
+			(at 62.23 159.6958 90)
 			(effects
 				(font
@@
 		)
 	)
-	(global_label "Q3"
+	(global_label "S3"
 		(shape input)
 		(at 72.39 165.1 90)
@@
 		)
 		(property "Intersheetrefs" "${INTERSHEET_REFS}"
-			(at 72.39 159.5748 90)
-			(effects
-				(font
-					(size 1.27 1.27)
-				)
-				(justify left)
-				(hide yes)
-			)
-		)
-	)
-	(global_label "Q2"
-		(shape input)
-		(at 62.23 165.1 90)
-		(fields_autoplaced yes)
-		(effects
-			(font
-				(size 1.27 1.27)
-			)
-			(justify left)
-		)
-		(property "Intersheetrefs" "${INTERSHEET_REFS}"
-			(at 62.23 159.5748 90)
+			(at 72.39 159.6958 90)
 			(effects
 				(font
@@
 		)
 	)
-	(global_label "Q1"
+	(global_label "S0"
+		(shape input)
+		(at 41.91 165.1 90)
+		(fields_autoplaced yes)
+		(effects
+			(font
+				(size 1.27 1.27)
+			)
+			(justify left)
+		)
+		(property "Intersheetrefs" "${INTERSHEET_REFS}"
+			(at 41.91 159.6958 90)
+			(effects
+				(font
+					(size 1.27 1.27)
+				)
+				(justify left)
+				(hide yes)
+			)
+		)
+	)
+	(global_label "S1"
 		(shape input)
 		(at 52.07 165.1 90)
@@
 		)
 		(property "Intersheetrefs" "${INTERSHEET_REFS}"
-			(at 52.07 159.5748 90)
+			(at 52.07 159.6958 90)
 			(effects
 				(font

Commit message: Daily sync 2025-08-30 21:30
Parts:
- D1, D3, D4, D5, D6: footprint LED_THT:LED_D3.0mm_Clear -> LED_SMD:LED_0805_2012Metric; Manufacturer Part No L-934GD -> KP-2012MGC
- D2: footprint LED_THT:LED_D3.0mm_Clear -> LED_SMD:LED_0805_2012Metric; Manufacturer Part No L-934ND -> KP-2012SECK
Changed lines of the file:
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@@
 			)
 		)
-		(property "Footprint" "LED_THT:LED_D3.0mm_Clear"
+		(property "Footprint" "LED_SMD:LED_0805_2012Metric"
 			(at 21.59 168.91 0)
 			(effects
@@
 			)
 		)
-		(property "Description" "LED, Low Power, Green, Through Hole, T-1 (3mm), 20 mA, 2.2 V, 568 nm"
+		(property "Description" "LED, Low Power, Green, SMD, 0805 [2012 Metric], 20 mA, 2.1 V, 570 nm"
 			(at 21.59 168.91 0)
 			(effects
@@
 			)
 		)
-		(property "Manufacturer Part No" "L-934GD"
+		(property "Manufacturer Part No" "KP-2012MGC"
 			(at 21.59 168.91 90)
 			(effects
@@
 			)
 		)
-		(property "Footprint" "LED_THT:LED_D3.0mm_Clear"
+		(property "Footprint" "LED_SMD:LED_0805_2012Metric"
 			(at 72.39 168.91 0)
 			(effects
@@
 			)
 		)
-		(property "Description" "LED, Low Power, Green, Through Hole, T-1 (3mm), 20 mA, 2.2 V, 568 nm"
+		(property "Description" "LED, Low Power, Green, SMD, 0805 [2012 Metric], 20 mA, 2.1 V, 570 nm"
 			(at 72.39 168.91 0)
 			(effects
@@
 			)
 		)
-		(property "Manufacturer Part No" "L-934GD"
+		(property "Manufacturer Part No" "KP-2012MGC"
 			(at 72.39 168.91 90)
 			(effects
@@
 			)
 		)
-		(property "Footprint" "LED_THT:LED_D3.0mm_Clear"
+		(property "Footprint" "LED_SMD:LED_0805_2012Metric"
 			(at 62.23 168.91 0)
 			(effects
@@
 			)
 		)
-		(property "Description" "LED, Low Power, Green, Through Hole, T-1 (3mm), 20 mA, 2.2 V, 568 nm"
+		(property "Description" "LED, Low Power, Green, SMD, 0805 [2012 Metric], 20 mA, 2.1 V, 570 nm"
 			(at 62.23 168.91 0)
 			(effects
@@
 			)
 		)
-		(property "Manufacturer Part No" "L-934GD"
+		(property "Manufacturer Part No" "KP-2012MGC"
 			(at 62.23 168.91 90)
 			(effects
@@
 			)
 		)
-		(property "Footprint" "LED_THT:LED_D3.0mm_Clear"
+		(property "Footprint" "LED_SMD:LED_0805_2012Metric"
 			(at 41.91 168.91 0)
 			(effects
@@
 			)
 		)
-		(property "Description" "LED, Low Power, Green, Through Hole, T-1 (3mm), 20 mA, 2.2 V, 568 nm"
+		(property "Description" "LED, Low Power, Green, SMD, 0805 [2012 Metric], 20 mA, 2.1 V, 570 nm"
 			(at 41.91 168.91 0)
 			(effects
@@
 			)
 		)
-		(property "Manufacturer Part No" "L-934GD"
+		(property "Manufacturer Part No" "KP-2012MGC"
 			(at 41.91 168.91 90)
 			(effects
@@
 			)
 		)
-		(property "Footprint" "LED_THT:LED_D3.0mm_Clear"
+		(property "Footprint" "LED_SMD:LED_0805_2012Metric"
 			(at 31.75 168.91 0)
 			(effects
@@
 			)
 		)
-		(property "Description" "LED, Low Power, Orange, Through Hole, T-1 (3mm), 20 mA, 2.05 V, 610 nm"
+		(property "Description" "LED, Low Power, Orange, SMD, 0805 [2012 Metric], 20 mA, 2.1 V, 601 nm"
 			(at 31.75 168.91 0)
 			(effects
@@
 			)
 		)
-		(property "Manufacturer Part No" "L-934ND"
+		(property "Manufacturer Part No" "KP-2012SECK"
 			(at 31.75 168.91 90)
 			(effects
@@
 			)
 		)
-		(property "Footprint" "LED_THT:LED_D3.0mm_Clear"
+		(property "Footprint" "LED_SMD:LED_0805_2012Metric"
 			(at 52.07 168.91 0)
 			(effects
@@
 			)
 		)
-		(property "Description" "LED, Low Power, Green, Through Hole, T-1 (3mm), 20 mA, 2.2 V, 568 nm"
+		(property "Description" "LED, Low Power, Green, SMD, 0805 [2012 Metric], 20 mA, 2.1 V, 570 nm"
 			(at 52.07 168.91 0)
 			(effects
@@
 			)
 		)
-		(property "Manufacturer Part No" "L-934GD"
+		(property "Manufacturer Part No" "KP-2012MGC"
 			(at 52.07 168.91 90)
 			(effects

Commit message: Daily sync 2025-08-31 12:14
Parts:
- removed D7: LED_Dual_AAK, LED_THT:LED_D3.0mm-3, symbol Device:LED_Dual_AAK
- added D7: AAA3528ESGCT, LED_SMD:AAA3528ESGCT, symbol Device:AAA3528ESGCT
Connections:
- net GND: now also D7.1 (K_RED), D7.3 (K_GREEN)
- net at R7.1: now also D7.2 (A_RED)
- net at R8.1: now also D7.4 (A_GREEN)
Other:
- moved on the sheet: C1, C2, C3, R7, R8

Commit message: Daily sync 2025-09-01 09:07
Other:
- moved on the sheet: C1, C2, C3, D1, D2, D3, D4, D5, D6, D7, R1, R2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
