File: PinCheck-4/PinCheck-4.kicad_pcb (KiCad board)
At the start: 2 copper layers, 61 parts, among them J1 Conn_01x02_Pin, J2 DA15_Socket, J3 LEMHAL Header, Q1 PMOS, SW1 SW_SPST, SW2 SW_SPST, U1 TPS61221DCK, U10 7408, U11 7432, U2 ICM7555xB, U3 4017, U4 TMUX1574DYY, U5 74HC14, U6 74HC14, U7 USBLC6-4SC6, U8 7408, U9 7432

Commit message: Daily sync 2025-08-28 16:55
Parts:
- removed C16: 100n, Capacitor_SMD:C_0805_2012Metric
- removed U11: 7432, Package_SO:SOIC-14_3.9x8.7mm_P1.27mm
- J1: moved to B.Cu
- U10: value 7408 -> 4072
- U9: value 7432 -> 7408
- moved U10 75.2 mm to (170.5, 60.3)
- moved J1 68.8 mm to (164.5, 81.7), turned to 90 degrees
- moved C15 65.7 mm to (151.6, 73.0)
- moved C13 53.4 mm to (151.6, 66.9)
- moved C14 53.4 mm to (151.6, 69.9)
- moved U8 53.4 mm to (153.6, 60.3)
- moved U9 53.4 mm to (162.1, 60.3)
- moved U5 46.5 mm to (163.1, 116.0)
- moved U6 46.5 mm to (171.6, 116.0)
- moved R16 44.6 mm to (172.8, 95.1)
- moved R17 44.6 mm to (172.8, 98.1)
- moved R18 44.6 mm to (172.8, 101.0)
- moved R19 44.6 mm to (172.8, 104.0)
- moved SW1 37.6 mm to (108.2, 102.9), turned to -90 degrees
- moved C11 28.8 mm to (177.3, 95.2)
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Connections:
- U10 pad 1: Q0 -> G
- U10 pad 10: NOT_S2 -> Net-(U10-Pad10)
- U10 pad 11: R3 -> Net-(U10-Pad11)
- U10 pad 12: Q3 -> Net-(U10-Pad12)
- U10 pad 13: NOT_S3 -> R
- U10 pad 2: NOT_S0 -> Net-(U10-Pad2)
- U10 pad 3: R0 -> Net-(U10-Pad3)
- U10 pad 4: Q1 -> Net-(U10-Pad4)
- U10 pad 5: NOT_S1 -> Net-(U10-Pad5)
- U10 pad 6: R1 -> (no net)
- U10 pad 8: R2 -> (no net)
- U10 pad 9: Q2 -> Net-(U10-Pad9)
- U8 pad 11: G3 -> Net-(U10-Pad5)
- U8 pad 3: G0 -> Net-(U10-Pad2)
- U8 pad 6: G1 -> Net-(U10-Pad3)
- U8 pad 8: G2 -> Net-(U10-Pad4)
- U9 pad 1: G0 -> Q0
- U9 pad 10: M2 -> NOT_S2
- U9 pad 11: unconnected-(U9-Pad11) -> Net-(U10-Pad12)
- U9 pad 12: unconnected-(U9-Pad12) -> Q3
- U9 pad 13: unconnected-(U9-Pad13) -> NOT_S3
- U9 pad 2: G1 -> NOT_S0
- U9 pad 3: M1 -> Net-(U10-Pad9)
- U9 pad 4: G2 -> Q1
- U9 pad 5: G3 -> NOT_S1
- U9 pad 6: M2 -> Net-(U10-Pad10)
- U9 pad 8: G -> Net-(U10-Pad11)
- U9 pad 9: M1 -> Q2
Other:
- board outline added: 25 x 70 mm

Commit message: Daily sync 2025-08-29 22:48
Parts:
- C10, C11, C12, C4, C5, C9, L1, Q1, R1, R11, R12, R13, R14, R15, R2, R3, R4, R5, R6, U1, U3, U4, U5, U6: moved to B.Cu
- D2: value LED -> Y LED
- J1: value Conn_01x02_Pin -> BatteryHolder
- J2: footprint Connector_Dsub:DSUB-15_Socket_Horizontal_P2.77x2.54mm_EdgePinOffset9.40mm -> Connector_Dsub:DSUB-15_Socket_Horizontal_P2.77x2.84mm_EdgePinOffset9.90mm_Housed_MountingHolesOffset11.32mm
- moved SW1 63.0 mm to (168.1, 122.0)
- moved C5 54.4 mm to (161.9, 129.8)
- moved C4 53.8 mm to (161.9, 122.7)
- moved Q1 49.7 mm to (161.9, 119.3), turned to 180 degrees
- moved C9 46.3 mm to (166.2, 74.0), turned to -90 degrees
- moved U10 46.2 mm to (157.9, 104.8), turned to -90 degrees
- moved R14 45.3 mm to (152.3, 76.3), turned to 90 degrees
- moved U3 45.2 mm to (159.4, 76.0), turned to 90 degrees
- moved C12 44.0 mm to (139.6, 120.9)
- moved R13 42.6 mm to (150.2, 76.3), turned to 90 degrees
- moved J3 40.7 mm to (148.0, 117.2)
- moved R11 39.8 mm to (148.1, 76.3), turned to 90 degrees
- moved U7 39.4 mm to (139.9, 129.0), turned to -90 degrees
- moved C11 39.3 mm to (147.6, 120.9)
- moved R17 39.2 mm to (143.7, 124.4)
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Other:
- board size 25 x 70 mm -> 39.2 x 60 mm

Commit message: Daily sync 2025-08-30 13:49
Parts:
- removed SW2: SW_SPST, Button_Switch_THT:SW_DIP_SPSTx01_Slide_9.78x4.72mm_W7.62mm_P2.54mm
- added REF**: ESD-Logo_6.6x6mm_SilkScreen, Symbol:ESD-Logo_6.6x6mm_SilkScreen, F.Cu at (151.8, 105.1)
- added SW3: OS102011MA1QS1, Button_Switch_THT:OS102011MA1QS1, F.Cu at (135.3, 123.1)
- added U1: MAX16054AZT_T, Package_TO_SOT_SMD:TSOT-23-6_HandSoldering, F.Cu at (167.6, 119.4)
- R7, R8: moved to B.Cu
- SW1: footprint Button_Switch_THT:SW_DIP_SPSTx01_Slide_9.78x4.72mm_W7.62mm_P2.54mm -> Button_Switch_THT:SW_PUSH_6mm
- moved C15 17.2 mm to (160.7, 89.9), turned to 180 degrees
- moved D7 16.8 mm to (167.4, 106.0)
- moved R8 9.72 mm to (164.9, 102.8), turned to 90 degrees
- moved R7 9.31 mm to (169.8, 102.8), turned to 90 degrees
- moved U10 8.69 mm to (167.2, 96.3)
- moved C14 8.69 mm to (169.2, 90.0)
- moved U11 8.56 mm to (158.7, 96.3), turned to 0 degrees
- moved C3 8.25 mm to (161.5, 121.5)
- moved C2 6.71 mm to (161.5, 119.3)
- moved R19 6.44 mm to (143.8, 123.8)
- moved R18 5.74 mm to (143.8, 121.6)
- moved C1 5.17 mm to (161.5, 117.0)
- moved R17 5.04 mm to (143.8, 119.3)
- moved R16 4.34 mm to (143.8, 117.1)
- moved RV1 4.32 mm to (142.8, 91.2)
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- renumbered U9 to U10, U10 to U11, U1 to U2, U2 to U3, U3 to U4, U4 to U5, U5 to U6, U6 to U7, U7 to U8, U8 to U9
Connections:
- J1 pad 1: Net-(J1-Pin_1) -> +BATT
- SW1 pad 1: Net-(J1-Pin_1) -> GND
- SW1 pad 2: Net-(Q1-S) -> Net-(SW1-B)
Routing:
- added copper zone on B.Cu, net GND
- added copper zone on F.Cu, net GND

Commit message: Daily sync 2025-08-30 21:30
Parts:
- removed REF**: ESD-Logo_6.6x6mm_SilkScreen, Symbol:ESD-Logo_6.6x6mm_SilkScreen
- C1, C13, C14, C15, C2, C3, C6, C7, R10, R9, U10, U11, U3, U9: moved to B.Cu
- D1, D2, D3, D4, D5, D6: footprint LED_THT:LED_D3.0mm_Clear -> LED_SMD:LED_0805_2012Metric
- J1: moved to F.Cu
- SW1: footprint Button_Switch_THT:SW_PUSH_6mm -> Button_Switch_SMD:SW_SPST_PTS645Sx43SMTR92
- moved SW2 43.4 mm to (168.8, 95.4), turned to 90 degrees
- moved R6 38.4 mm to (136.1, 129.4), turned to 0 degrees
- moved D6 35.7 mm to (136.1, 129.4), turned to 0 degrees
- moved D1 34.4 mm to (169.6, 114.8)
- moved R1 34.3 mm to (169.6, 114.8), turned to 90 degrees
- moved R5 31.5 mm to (136.1, 126.8), turned to 0 degrees
- moved C14 31.0 mm to (140.8, 102.6), turned to 0 degrees
- moved D5 28.6 mm to (136.1, 126.8), turned to 0 degrees
- moved U10 27.4 mm to (142.8, 108.8), turned to 180 degrees
- moved C3 26.6 mm to (136.0, 114.1)
- moved C2 25.7 mm to (136.0, 116.3)
- moved C1 25.5 mm to (136.0, 118.6)
- moved R4 24.5 mm to (136.1, 124.3), turned to 0 degrees
- moved D4 21.5 mm to (136.1, 124.3), turned to 0 degrees
- moved D7 20.4 mm to (154.1, 90.6)
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- renumbered SW3 to SW2
Connections:
- D3 pad 2: Q0 -> S0
- D4 pad 2: Q1 -> S1
- D5 pad 2: Q2 -> S2
- D6 pad 2: Q3 -> S3

Commit message: Daily sync 2025-08-31 12:14
Parts:
- added G***: LOGO, Symbol:akuray logo (miniature), B.Cu at (140.6, 74.4)
- added G***: LOGO, Symbol:akuray (miniature), B.Cu at (146.9, 74.0)
- added G***: LOGO, Symbol:Hand logo 10x10, B.Cu at (135.6, 75.5)
- C1, C10, C2, C3, C4, C5, L1, Q1, R1, R15, U2, U5: moved to F.Cu
- D7: value LED_Dual_AAK -> AAA3528ESGCT; footprint LED_THT:LED_D3.0mm-3 -> LED_SMD:AAA3528ESGCT
- R16, R17, R18, R19, U8: moved to B.Cu
- moved D7 35.1 mm to (141.2, 123.2), turned to -90 degrees
- moved R7 29.8 mm to (134.8, 117.2), turned to 180 degrees
- moved R8 28.8 mm to (134.8, 119.7), turned to 180 degrees
- moved R15 28.5 mm to (155.7, 91.4), turned to 0 degrees
- moved R12 28.2 mm to (159.6, 99.6), turned to 180 degrees
- moved R11 24.9 mm to (159.6, 97.1), turned to 180 degrees
- moved C9 23.2 mm to (150.7, 88.5), turned to 0 degrees
- moved R13 21.7 mm to (159.6, 94.7), turned to 180 degrees
- moved U4 21.6 mm to (152.7, 95.6), turned to 180 degrees
- moved U5 19.6 mm to (151.4, 90.0)
- moved R14 18.6 mm to (159.6, 92.3), turned to 180 degrees
- moved C10 18.1 mm to (155.8, 88.5), turned to 0 degrees
- moved D1 17.4 mm to (160.0, 129.3), turned to 0 degrees
- moved R1 15.4 mm to (159.9, 126.7), turned to 0 degrees
- moved L1 15.0 mm to (168.3, 111.1), turned to 180 degrees
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Connections:
- D7 pad 1: Net-(D7-A1) -> GND
- D7 pad 2: Net-(D7-A2) -> Net-(D7-A_RED)
- R7 pad 1: Net-(D7-A1) -> Net-(D7-A_RED)
- R8 pad 1: Net-(D7-A2) -> Net-(D7-A_GREEN)
Other:
- board text added: "CCBFH-ISO-DB15H4P3525.01"
- board text added: "IGBT"
- board text added: "OVP"
- board text added: "SINGNAL MONITOR"

Commit message: Daily sync 2025-08-31 16:37
Parts:
- moved D1 12.3 mm to (166.9, 119.1), turned to 90 degrees
- moved R1 11.9 mm to (169.1, 119.1), turned to 90 degrees
- moved Q1 7.50 mm to (164.0, 109.8)
- moved U1 3.16 mm to (160.4, 119.1), turned to 0 degrees
- moved SW1 3.02 mm to (163.9, 126.1)
- moved C4 2.77 mm to (163.5, 113.3)
- moved C5 2.67 mm to (169.5, 113.3)
- moved L1 2.34 mm to (168.7, 108.8)
- moved U2 2.21 mm to (166.5, 113.6)
- moved D3 0.94 mm to (135.5, 119.1)
- moved D5 0.94 mm to (135.5, 125.5)
- moved D6 0.94 mm to (135.5, 128.7)
- moved D4 0.94 mm to (135.5, 122.3)
- moved D7 0.89 mm to (142.1, 123.5)
- moved J3 0.25 mm to (147.7, 117.2)
Other:
- outline, holes or cut-outs redrawn
- board text added: "--.-POWER........."
- board text added: "MODE SELECTION"

Commit message: Daily sync 2025-09-01 11:59
Parts:
- removed J3: LEMHAL Header, Connector_Molex:SHDRRA4W70P0X254_1X4_1016X1170X580P
- added BT1: 1070TR, Connector:KEYSTONE_1070TR, F.Cu at (149.1, 103.8)
- J1: value BatteryHolder -> DA15_Socket; footprint Battery:BatteryHolder_Keystone_1060_1x2032 -> Connector_Dsub:DSUB-15_Socket_Horizontal_P2.77x2.84mm_EdgePinOffset9.90mm_Housed_MountingHolesOffset11.32mm
- J2: value DA15_Socket -> LEMHAL Header; footprint Connector_Dsub:DSUB-15_Socket_Horizontal_P2.77x2.84mm_EdgePinOffset9.90mm_Housed_MountingHolesOffset11.32mm -> Connector:CONN_A-7478-04A_MOL
- moved J2 33.9 mm to (147.7, 118.1), turned to 0 degrees
- moved J1 21.3 mm to (141.8, 84.7)
- moved RV1 14.4 mm to (134.7, 103.0)
- moved C5 8.51 mm to (161.0, 113.5), turned to 90 degrees
- moved L1 4.97 mm to (168.5, 113.8)
- moved Q1 4.96 mm to (169.0, 109.2)
- moved C4 4.50 mm to (159.0, 113.5), turned to -90 degrees
- moved U2 2.11 mm to (164.4, 113.8)
- moved C8 0.10 mm to (135.1, 91.4)
Connections:
- J1 pad 1: +BATT -> unconnected-(J1-Pad1)
- J1 pad 2: GND -> Net-(U5-S1A)
- J2 pad 1: unconnected-(J2-Pad1) -> Net-(U8-I/O1)
- J2 pad 2: Net-(U5-S1A) -> Net-(U8-I/O2)
- J2 pad 3: Net-(U5-S1B) -> Net-(U8-I/O3)
- J2 pad 4: Net-(U5-S2B) -> Net-(U8-I/O4)
- R16 pad 1: Net-(J3-Pin_1) -> Net-(U8-I/O1)
- R17 pad 1: Net-(J3-Pin_2) -> Net-(U8-I/O2)
- R18 pad 1: Net-(J3-Pin_3) -> Net-(U8-I/O3)
- R19 pad 1: Net-(J3-Pin_4) -> Net-(U8-I/O4)
- U5 pad 10: Net-(J2-P10) -> Net-(J1-P10)
- U5 pad 11: Net-(J2-P9) -> Net-(J1-P9)
- U5 pad 13: Net-(J2-P111) -> Net-(J1-P111)
- U5 pad 14: Net-(J2-P10) -> Net-(J1-P10)
- U6 pad 1: Net-(J3-Pin_1) -> Net-(U8-I/O1)
- U6 pad 3: Net-(J3-Pin_2) -> Net-(U8-I/O2)
- U6 pad 5: Net-(J3-Pin_3) -> Net-(U8-I/O3)
- U6 pad 9: Net-(J3-Pin_4) -> Net-(U8-I/O4)
- U8 pad 1: Net-(J3-Pin_1) -> Net-(U8-I/O1)
- U8 pad 3: Net-(J3-Pin_2) -> Net-(U8-I/O2)
- U8 pad 4: Net-(J3-Pin_3) -> Net-(U8-I/O3)
- U8 pad 6: Net-(J3-Pin_4) -> Net-(U8-I/O4)
