File: PinCheck-4/PinCheck-4.kicad_pcb (KiCad board)
At the start: 2 copper layers, 39.2 x 60 mm, 63 parts, among them J1 DA15_Socket, J2 LEMHAL Header, Q1 PMOS, SW1 SW_SPST, SW2 OS102011MA1QS1, U1 MAX16054AZT_T, U10 7408, U11 4072, U2 TPS61221DCK, U3 ICM7555xB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

Commit message: Daily sync 2025-09-16 16:52
Parts:
- moved R12 7.22 mm to (159.6, 92.3), turned to 0 degrees
- moved R14 7.22 mm to (159.6, 99.6), turned to 0 degrees
- moved R11 2.41 mm to (159.6, 94.7), turned to 0 degrees
- moved R13 2.41 mm to (159.6, 97.1), turned to 0 degrees
Routing:
- net S2: track 0.00 -> 81.0 mm, vias 0 -> 4
- net Net-(U8-I/O4): track 0.00 -> 77.5 mm, vias 0 -> 1
- net Net-(U8-I/O2): track 0.00 -> 75.2 mm, vias 0 -> 3
- net S0: track 0.00 -> 65.3 mm, vias 0 -> 3
- net Net-(U8-I/O1): track 0.00 -> 55.1 mm, vias 0 -> 3
- net S1: track 0.00 -> 54.8 mm, vias 0 -> 2
- net S3: track 0.00 -> 51.1 mm, vias 0 -> 3
- net Net-(U8-I/O3): track 0.00 -> 48.1 mm, vias 0 -> 2
- net NOT_S0: track 0.00 -> 38.4 mm, vias 0 -> 2
- net NOT_S2: track 0.00 -> 34.7 mm, vias 0 -> 2
- net NOT_S1: track 0.00 -> 33.3 mm, vias 0 -> 2
- net Q2: track 0.00 -> 32.1 mm, vias 0 -> 2
- net G: track 0.00 -> 29.4 mm, vias 0 -> 2
- net NOT_S3: track 0.00 -> 28.9 mm, vias 0 -> 2
- net Q3: track 0.00 -> 28.8 mm, vias 0 -> 2
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- added copper zone on In1.Cu, net GND
- added copper zone on B.Cu, net VCC
- added copper zone on F.Cu, net VCC
- added copper zone on In2.Cu, net VCC
Other:
- copper layers 2 -> 4

Commit message: Daily sync 2025-09-17 12:09
Parts:
- added REF**: ESD-Logo_6.6x6mm_SilkScreen, Symbol:ESD-Logo_6.6x6mm_SilkScreen, B.Cu at (167.2, 75.1)
Routing:
- net Q1: track 3.54 -> 55.3 mm, vias 0 -> 3
- net Q0: track 3.97 -> 46.0 mm, vias 0 -> 4
- net Net-(J1-P111): track 0.00 -> 34.7 mm, vias 0 -> 1
- net Net-(J1-P9): track 0.00 -> 30.9 mm, vias 0 -> 1
- net Net-(SW2-COM): track 0.00 -> 27.5 mm, vias 0 -> 3
- net Q2: track 32.1 -> 54.3 mm, vias 2 -> 3
- net Q3: track 28.8 -> 49.4 mm, vias 2 -> 3
- net Net-(U5-D2): track 0.00 -> 19.4 mm, vias 0 -> 2
- net Net-(U5-D1): track 0.00 -> 19.4 mm, vias 0 -> 1
- net Net-(U5-D4): track 0.00 -> 18.8 mm, vias 0 -> 3
- net Net-(J1-P10): track 0.00 -> 18.3 mm, vias 0 -> 1
- net Net-(U5-S2B): track 0.00 -> 16.6 mm, vias 0 -> 1
- net Net-(U5-D3): track 0.00 -> 10.8 mm, vias 0 -> 1
- net Net-(U5-S1B): track 0.00 -> 10.1 mm
- net Net-(U4-Q4): track 0.00 -> 8.55 mm
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Other:
- board text added: "CCBFH-ISO-DB15H4P3825.01"
- board text removed: "CCBFH-ISO-DB15H4P3525.01"

Commit message: Daily sync 2025-09-17 15:01
Other:
- board text added: "CBFH-ISO-DB15H4P3825.01"
- board text removed: "CCBFH-ISO-DB15H4P3825.01"
Changed lines of the file:
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@@
 		)
 	)
-	(gr_text "CCBFH-ISO-DB15H4P3825.01"
+	(gr_text "CBFH-ISO-DB15H4P3825.01"
 		(at 139.323873 72.119948 180)
 		(layer "B.SilkS")
