File: PinCheck-4/clock_logic.kicad_sch (KiCad schematic)
At the start: 24 parts, among them J1 DB9 In, U1 NE555D, U2 4017

Commit message: Daily sync 2025-08-27 16:57
Parts:
- removed C2: 100n, symbol Device:C
- removed D1, D2, D3, D4, D5: LED, symbol Device:LED
- removed J1: DB9 In, symbol Connector:Conn_01x04_Socket
- removed R1, R10, R3, R4, R5, R6, R7, R8, R9: 1k, symbol Device:R
- removed U1: NE555D, Package_SO:SOIC-8_3.9x4.9mm_P1.27mm, symbol Timer:NE555D
- removed U2: 4017, symbol 4xxx:4017
- added C4, C5: 10u, Capacitor_SMD:C_0805_2012Metric, symbol Device:C
- added J1: Conn_01x02_Pin, Battery:BatteryHolder_Keystone_1060_1x2032, symbol Connector:Conn_01x02_Pin
- added L1: 4.7u, Inductor_SMD:EPL3015472MLC, symbol Device:L
- added Q1: PMOS, Package_TO_SOT_SMD:SOT-323_SC-70, symbol Simulation_SPICE:PMOS
- added SW1: SW_SPST, Button_Switch_THT:SW_DIP_SPSTx01_Slide_9.78x4.72mm_W7.62mm_P2.54mm, symbol Switch:SW_SPST
- added U1: TPS61221DCK, Package_TO_SOT_SMD:Texas_R-PDSO-G6, symbol Regulator_Switching:TPS61221DCK
- added U2: ICM7555xB, Package_SO:SOIC-8_3.9x4.9mm_P1.27mm, symbol Timer:ICM7555xB
- C6: renamed from C1; footprint (none) -> Capacitor_SMD:C_0805_2012Metric
- C7: renamed from C4; footprint (none) -> Capacitor_SMD:C_0805_2012Metric
- C8: renamed from C6; footprint (none) -> Capacitor_SMD:CP_Elec_5x4.5
- R10: renamed from R2; footprint (none) -> Resistor_SMD:R_0805_2012Metric
- R9: renamed from R17; footprint (none) -> Resistor_SMD:R_0805_2012Metric
- RV1: footprint (none) -> Potentiometer_SMD:Potentiometer_Bourns_3314G_Vertical
Connections:
- net CLK: now also U2.3 (Q)
- net GND: now also C4.2, C5.2, J1.2 (Pin_2), Q1.1 (G), U1.3 (GND), U2.1 (GND)
- net VCC: now also C5.1, U1.2 (FB), U1.4 (VOUT), U2.4 (R), U2.8 (VCC)
- net at C7.1: now also U2.5 (CV)
- net at C8.1, R9.1: now also U2.2 (TR), U2.6 (THR)
- net at R10.2, R9.2: now also U2.7 (DIS)
- new net: C4.1, L1.1, Q1.3 (D), U1.1 (VIN), U1.6 (EN)
- new net: Q1.2 (S), SW1.2 (B)
- new net: J1.1 (Pin_1), SW1.1 (A)
- new net: L1.2, U1.5 (L)
Other:
- note added: "Use CMOS 555 for ultra low current such as TLC555 or 7555"
- note removed: "ADD a selector to change DB9 as per mode TOP / BOTTOM (IGBT & OVP)"
- moved on the sheet: C6, C7, C8, R10, R9, RV1

Commit message: Daily sync 2025-08-28 16:55
Changed lines of the file:
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@@
 	)
 	(junction
-		(at 105.41 99.06)
+		(at 78.74 99.06)
 		(diameter 0)
 		(color 0 0 0 0)
@@
 	(wire
 		(pts
-			(xy 105.41 96.52) (xy 105.41 99.06)
-		)
-		(stroke
-			(width 0)
-			(type default)
-		)
-	)
-	(wire
-		(pts
 			(xy 256.54 86.36) (xy 259.08 86.36)
 		)
@@
 	(wire
 		(pts
-			(xy 105.41 99.06) (xy 114.3 99.06)
-		)
-		(stroke
-			(width 0)
-			(type default)
-		)
-	)
-	(wire
-		(pts
 			(xy 78.74 104.14) (xy 78.74 101.6)
 		)
@@
 	(wire
 		(pts
-			(xy 105.41 99.06) (xy 101.6 99.06)
+			(xy 101.6 99.06) (xy 114.3 99.06)
 		)
 		(stroke
@@
 	(wire
 		(pts
-			(xy 77.47 99.06) (xy 81.28 99.06)
+			(xy 77.47 99.06) (xy 78.74 99.06)
+		)
+		(stroke
+			(width 0)
+			(type default)
+		)
+	)
+	(wire
+		(pts
+			(xy 78.74 82.55) (xy 78.74 99.06)
 		)
 		(stroke
@@
 		(pts
 			(xy 238.76 101.6) (xy 238.76 109.22)
+		)
+		(stroke
+			(width 0)
+			(type default)
+		)
+	)
+	(wire
+		(pts
+			(xy 78.74 99.06) (xy 81.28 99.06)
 		)
 		(stroke
@@
 	)
 	(symbol
-		(lib_id "power:PWR_FLAG")
-		(at 105.41 96.52 0)
-		(unit 1)
-		(exclude_from_sim no)
-		(in_bom yes)
-		(on_board yes)
-		(dnp no)
-		(fields_autoplaced yes)
-		(property "Reference" "#FLG02"
-			(at 105.41 94.615 0)
-			(effects
-				(font
-					(size 1.27 1.27)
-				)
-				(hide yes)
-			)
-		)
-		(property "Value" "PWR_FLAG"
-			(at 105.41 91.44 0)
-			(effects
-				(font
-					(size 1.27 1.27)
-				)
-			)
-		)
-		(property "Footprint" ""
-			(at 105.41 96.52 0)
-			(effects
-				(font
-					(size 1.27 1.27)
-				)
-				(hide yes)
-			)
-		)
-		(property "Datasheet" "~"
-			(at 105.41 96.52 0)
-			(effects
-				(font
-					(size 1.27 1.27)
-				)
-				(hide yes)
-			)
-		)
-		(property "Description" "Special symbol for telling ERC where power comes from"
-			(at 105.41 96.52 0)
-			(effects
-				(font
-					(size 1.27 1.27)
-				)
-				(hide yes)
-			)
-		)
-		(pin "1"
-		)
-		(instances
-			(project "PinCheck-4"
-				(path "/8e21fa9a-50eb-4ff7-ab75-73c4d6c5f942/83536851-927e-4d27-972f-18188fbc94fe"
-					(reference "#FLG02")
-					(unit 1)
-				)
-			)
-		)
-	)
-	(symbol
 		(lib_id "power:GND")
 		(at 180.34 120.65 0)
@@
 					(unit 1)
 				)
+			)
+		)
+	)
+	(symbol
+		(lib_id "power:PWR_FLAG")
+		(at 78.74 82.55 0)
+		(unit 1)
+		(exclude_from_sim no)
+		(in_bom yes)
+		(on_board yes)
+		(dnp no)
+		(fields_autoplaced yes)
+		(property "Reference" "#FLG02"
+			(at 78.74 80.645 0)
+			(effects
+				(font
+					(size 1.27 1.27)
+				)
+				(hide yes)
+			)
+		)
+		(property "Value" "PWR_FLAG"
+			(at 78.74 77.47 0)
+			(effects
+				(font
+					(size 1.27 1.27)
+				)
+			)
+		)
+		(property "Footprint" ""
+			(at 78.74 82.55 0)
+			(effects
+				(font
+					(size 1.27 1.27)
+				)
+				(hide yes)
+			)
+		)
+		(property "Datasheet" "~"
+			(at 78.74 82.55 0)
+			(effects
+				(font
+					(size 1.27 1.27)
+				)
+				(hide yes)
+			)
+		)
+		(property "Description" "Special symbol for telling ERC where power comes from"
+			(at 78.74 82.55 0)
+			(effects
+				(font
+					(size 1.27 1.27)
+				)
+				(hide yes)
+			)
+		)
+		(pin "1"
+		)
+		(instances
+			(project ""
+				(path "/8e21fa9a-50eb-4ff7-ab75-73c4d6c5f942/83536851-927e-4d27-972f-18188fbc94fe"
+					(reference "#FLG02")
+					(unit 1)
+				)

Commit message: Daily sync 2025-08-29 22:48
Parts:
- C4, C5: Manufacturer Part No (none) -> C2012X5R1C106M085AC
- C6: Manufacturer Part No (none) -> 0805B104K160CT
- C7: Manufacturer Part No (none) -> C0805S103K4RACTU
- C8: Manufacturer Part No (none) -> EEE1EA4R7NR
- J1: value Conn_01x02_Pin -> BatteryHolder; Manufacturer Part No (none) -> 1057TR
- L1: Manufacturer Part No (none) -> EPL3015-472MLC
- Q1: Manufacturer Part No (none) -> AO3407A
- R10, R9: Manufacturer Part No (none) -> CR0805-FX-1002ELF
- RV1: Manufacturer Part No (none) -> 3314G-1-104E
- SW1: Manufacturer Part No (none) -> Dip Switch SPST 1 Position Through Hole Slide (Standard) Ac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
- U1: Manufacturer Part No (none) -> TPS61221DCKT
- U2: Manufacturer Part No (none) -> ICM7555ESA+T
Changed lines of the file:
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@@
 			)
 		)
-		(property "Description" "Unpolarized capacitor"
+		(property "Description" "SMD Multilayer Ceramic Capacitor, 10 µF, 16 V, 0805 [2012 Metric], ± 20%, X5R"
+			(at 67.31 109.22 0)
+			(effects
+				(font
+					(size 1.27 1.27)
+				)
+				(hide yes)
+			)
+		)
+		(property "Manufacturer Part No" "C2012X5R1C106M085AC"
 			(at 67.31 109.22 0)
 			(effects
@@
 			)
 		)
-		(property "Description" "P-MOSFET transistor, drain/source/gate"
+		(property "Description" "MOSFET P-CH 30V 4.3A SOT23-3L"
 			(at 64.77 88.9 0)
 			(effects
@@
 			)
 		)
+		(property "Manufacturer Part No" "AO3407A"
+			(at 64.77 88.9 0)
+			(effects
+				(font
+					(size 1.27 1.27)
+				)
+				(hide yes)
+			)
+		)
 		(pin "3"
 		)
@@
 			)
 		)
-		(property "Description" "Unpolarized capacitor"
+		(property "Description" "SMD Multilayer Ceramic Capacitor, 0.1 µF, 16 V, 0805 [2012 Metric], ± 10%, X7R"
+			(at 180.34 86.36 0)
+			(effects
+				(font
+					(size 1.27 1.27)
+				)
+				(hide yes)
+			)
+		)
+		(property "Manufacturer Part No" "0805B104K160CT"
 			(at 180.34 86.36 0)
 			(effects
@@
 			)
 		)
-		(property "Description" "Unpolarized capacitor"
+		(property "Description" "SMD Multilayer Ceramic Capacitor, 0.01 µF, 16 V, 0805 [2012 Metric], ± 10%, X7R"
+			(at 180.34 114.3 0)
+			(effects
+				(font
+					(size 1.27 1.27)
+				)
+				(hide yes)
+			)
+		)
+		(property "Manufacturer Part No" "C0805S103K4RACTU"
 			(at 180.34 114.3 0)
 			(effects
@@
 			)
 		)
-		(property "Description" "Single Pole Single Throw (SPST) switch"
+		(property "Description" "Dip Switch SPST 1 Position Through Hole Slide (Standard) Actuator 25mA 24VDC"
+			(at 55.88 78.74 0)
+			(effects
+				(font
+					(size 1.27 1.27)
+				)
+				(hide yes)
+			)
+		)
+		(property "Manufacturer Part No" "Dip Switch SPST 1 Position Through Hole Slide (Standard) Actuator 25mA 24VDC"
 			(at 55.88 78.74 0)
 			(effects
@@
 			)
 		)
-		(property "Description" "CMOS General Purpose Timer, 555 compatible, SOIC-8"
+		(property "Description" "555 Type, Timer/Oscillator (Single) IC 500kHz 8-SOIC"
+			(at 212.09 109.22 0)
+			(effects
+				(font
+					(size 1.27 1.27)
+				)
+				(hide yes)
+			)
+		)
+		(property "Manufacturer Part No" "ICM7555ESA+T"
 			(at 212.09 109.22 0)
 			(effects
@@
 			)
 		)
-		(property "Description" "Polarized capacitor"
+		(property "Description" "SMD Aluminium Electrolytic Capacitor, Radial Can - SMD, 4.7 µF, 25 V, 2000 hours @ 85°C"
+			(at 246.38 120.65 0)
+			(effects
+				(font
+					(size 1.27 1.27)
+				)
+				(hide yes)
+			)
+		)
+		(property "Manufacturer Part No" "EEE1EA4R7NR"
 			(at 246.38 120.65 0)
 			(effects
@@
 			)
 		)
-		(property "Value" "Conn_01x02_Pin"
+		(property "Value" "BatteryHolder"
 			(at 36.83 76.454 0)
 			(effects
@@
 			)
 		)
-		(property "Description" "Generic connector, single row, 01x02, script generated"
+		(property "Description" "Battery Holder (Open) Coin, 20.0mm 1 Cell SMD (SMT) Tab"
+			(at 36.83 78.74 0)
+			(effects
+				(font
+					(size 1.27 1.27)
+				)
+				(hide yes)
+			)
+		)
+		(property "Manufacturer Part No" "1057TR"
 			(at 36.83 78.74 0)
 			(effects
@@
 			)
 		)
-		(property "Description" "Resistor"
+		(property "Description" "SMD Chip Resistor, 10 kohm, ± 1%, 125 mW, 0805 [2012 Metric], Thick Film, General Purpose"
+			(at 252.73 97.79 0)
+			(effects
+				(font
+					(size 1.27 1.27)
+				)
+				(hide yes)
+			)
+		)
+		(property "Manufacturer Part No" "CR0805-FX-1002ELF"
 			(at 252.73 97.79 0)
 			(effects
@@
 			)
 		)
+		(property "Manufacturer Part No" "TPS61221DCKT "
+			(at 91.44 101.6 0)
+			(effects
+				(font
+					(size 1.27 1.27)
+				)
+				(hide yes)
+			)
+		)
 		(pin "1"
 		)
@@
 			)
 		)
-		(property "Description" "Inductor"
+		(property "Description" "Power Inductor (SMD), 4.7 µH, 1.4 A, Shielded, 550 mA, EPL3015 Series"
 			(at 73.66 99.06 0)
+			(effects
+				(font
+					(size 1.27 1.27)
+				)
+				(hide yes)
+			)
+		)
+		(property "Manufacturer Part No" "EPL3015-472MLC"
+			(at 73.66 99.06 90)
 			(effects
 				(font
@@
 			)
 		)
-		(property "Description" "Unpolarized capacitor"
+		(property "Description" "SMD Multilayer Ceramic Capacitor, 10 µF, 16 V, 0805 [2012 Metric], ± 20%, X5R"
+			(at 114.3 109.22 0)
+			(effects
+				(font
+					(size 1.27 1.27)
+				)
+				(hide yes)
+			)
+		)
+		(property "Manufacturer Part No" "C2012X5R1C106M085AC"
 			(at 114.3 109.22 0)
 			(effects
@@
 			)
 		)
-		(property "Description" "Potentiometer"
+		(property "Description" "Trimmer, Single Turn, Cermet, Top Adjust, 100 kohm, Surface Mount, 1 Turns"
+			(at 252.73 86.36 0)
+			(effects
+				(font
+					(size 1.27 1.27)
+				)
+				(hide yes)
+			)
+		)
+		(property "Manufacturer Part No" "3314G-1-104E"
 			(at 252.73 86.36 0)
 			(effects
@@
 			)
 		)
-		(property "Description" "Resistor"
+		(property "Description" "SMD Chip Resistor, 10 kohm, ± 1%, 125 mW, 0805 [2012 Metric], Thick Film, General Purpose"
 			(at 238.76 97.79 0)
 			(effects
+				(font
+					(size 1.27 1.27)
+				)
+				(hide yes)
+			)
+		)
+		(property "Manufacturer Part No" "CR0805-FX-1002ELF"
+			(at 238.76 97.79 0)
+			(effects

Commit message: Daily sync 2025-08-30 13:49
Parts:
- added U1: MAX16054AZT_T, Package_TO_SOT_SMD:TSOT-23-6_HandSoldering, symbol Switch:MAX16054AZT_T
- SW1: footprint Button_Switch_THT:SW_DIP_SPSTx01_Slide_9.78x4.72mm_W7.62mm_P2.54mm -> Button_Switch_THT:SW_PUSH_6mm; Manufacturer Part No Dip Switch SPST 1 Position Through Hole Slide (Standard) Ac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 -> TS02-66-70-BK-260-LCR-D
- renumbered U1 to U2, U2 to U3
Connections:
- net GND: now also SW1.1 (A), U1.2 (GND), U1.3 (CLEAR)
- net at Q1.2 (S): now also U1.5 (OUT); no longer SW1.2 (B)
- net +BATT: now reaches J1.1 (Pin_1)
- net +BATT: now also U1.6 (VCC); no longer SW1.1 (A)
- new net: SW1.2 (B), U1.1 (IN)
- no-connect marks 0 -> 1
Other:
- moved on the sheet: C4, C5, J1, L1, Q1, SW1, U2

Commit message: Daily sync 2025-08-30 21:30
Parts:
- SW1: footprint Button_Switch_THT:SW_PUSH_6mm -> Button_Switch_SMD:SW_SPST_PTS645Sx43SMTR92; Manufacturer Part No TS02-66-70-BK-260-LCR-D -> TS04-66-70-BK-160-SMT
Changed lines of the file:
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@@
 			)
 		)
-		(property "Footprint" "Button_Switch_THT:SW_PUSH_6mm"
+		(property "Footprint" "Button_Switch_SMD:SW_SPST_PTS645Sx43SMTR92"
 			(at 36.83 93.98 0)
 			(effects
@@
 			)
 		)
-		(property "Description" "Tactile Switch SPST-NO Top Actuated Through Hole"
+		(property "Description" "TS04-66-70-BK-160-SMT"
 			(at 36.83 93.98 0)
 			(effects
@@
 			)
 		)
-		(property "Manufacturer Part No" "TS02-66-70-BK-260-LCR-D"
+		(property "Manufacturer Part No" "TS04-66-70-BK-160-SMT"
 			(at 36.83 93.98 0)
 			(effects

Commit message: Daily sync 2025-09-01 09:07
Other:
- note added: "Use CMOS TLC555 or 7555 for ultra low current"
- note removed: "Use CMOS 555 for ultra low current such as TLC555 or 7555"
- moved on the sheet: C4, C5, C6, C7, C8, J1, L1, Q1, R10, R9, RV1, SW1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

Commit message: Daily sync 2025-09-01 11:59
Parts:
- removed J1: BatteryHolder, Battery:BatteryHolder_Keystone_1060_1x2032, symbol Connector:Conn_01x02_Pin
- added BT1: 1070TR, Connector:KEYSTONE_1070TR, symbol PinCheck-4_Library:1070TR
Connections:
- net +BATT: now also BT1.P
- net GND: now also BT1.N
Changed lines of the file:
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@@
+	)
+	(junction
+		(at 91.44 74.93)
+		(diameter 0)
+		(color 0 0 0 0)
 	)
 	(junction
@@
 	)
 	(junction
-		(at 82.55 74.93)
-		(diameter 0)
-		(color 0 0 0 0)
-	)
-	(junction
 		(at 91.44 127)
 		(diameter 0)
@@
 	(wire
 		(pts
-			(xy 82.55 74.93) (xy 93.98 74.93)
-		)
-		(stroke
-			(width 0)
-			(type default)
-		)
-	)
-	(wire
-		(pts
-			(xy 91.44 77.47) (xy 93.98 77.47)
-		)
-		(stroke
-			(width 0)
-			(type default)
-		)
-	)
-	(wire
-		(pts
 			(xy 35.56 82.55) (xy 35.56 85.09)
 		)
@@
 	(wire
 		(pts
-			(xy 72.39 74.93) (xy 82.55 74.93)
+			(xy 72.39 74.93) (xy 91.44 74.93)
 		)
 		(stroke
@@
 	(wire
 		(pts
-			(xy 82.55 72.39) (xy 82.55 74.93)
-		)
-		(stroke
-			(width 0)
-			(type default)
-		)
-	)
-	(wire
-		(pts
-			(xy 91.44 77.47) (xy 91.44 83.82)
+			(xy 91.44 71.12) (xy 91.44 74.93)
+		)
+		(stroke
+			(width 0)
+			(type default)
+		)
+	)
+	(wire
+		(pts
+			(xy 91.44 90.17) (xy 91.44 91.44)
 		)
 		(stroke
@@
 	)
 	(symbol
+		(lib_id "PinCheck-4_Library:1070TR")
+		(at 91.44 82.55 270)
+		(unit 1)
+		(exclude_from_sim no)
+		(in_bom yes)
+		(on_board yes)
+		(dnp no)
+		(fields_autoplaced yes)
+		(property "Reference" "BT1"
+			(at 95.25 80.6449 90)
+			(effects
+				(font
+					(size 1.27 1.27)
+				)
+				(justify left)
+			)
+		)
+		(property "Value" "1070TR"
+			(at 95.25 83.1849 90)
+			(effects
+				(font
+					(size 1.27 1.27)
+				)
+				(justify left)
+			)
+		)
+		(property "Footprint" "Connector:KEYSTONE_1070TR"
+			(at 91.44 82.55 0)
+			(effects
+				(font
+					(size 1.27 1.27)
+				)
+				(justify bottom)
+				(hide yes)
+			)
+		)
+		(property "Datasheet" ""
+			(at 91.44 82.55 0)
+			(effects
+				(font
+					(size 1.27 1.27)
+				)
+				(hide yes)
+			)
+		)
+		(property "Description" "Battery Holder (Open) Coin, 20.0mm 1 Cell SMD (SMT) Tab"
+			(at 91.44 82.55 0)
+			(effects
+				(font
+					(size 1.27 1.27)
+				)
+				(hide yes)
+			)
+		)
+		(property "PARTREV" "C"
+			(at 91.44 82.55 0)
+			(effects
+				(font
+					(size 1.27 1.27)
+				)
+				(justify bottom)
+				(hide yes)
+			)
+		)
+		(property "STANDARD" "Manufacturer Recommendations"
+			(at 91.44 82.55 0)
+			(effects
+				(font
+					(size 1.27 1.27)
+				)
+				(justify bottom)
+				(hide yes)
+			)
+		)
+		(property "SNAPEDA_PN" "1070"
+			(at 91.44 82.55 0)
+			(effects
+				(font
+					(size 1.27 1.27)
+				)
+				(justify bottom)
+				(hide yes)
+			)
+		)
+		(property "MAXIMUM_PACKAGE_HEIGHT" "5.97mm"
+			(at 91.44 82.55 0)
+			(effects
+				(font
+					(size 1.27 1.27)
+				)
+				(justify bottom)
+				(hide yes)
+			)
+		)
+		(property "MANUFACTURER" "Keystone Electronics"
+			(at 91.44 82.55 0)
+			(effects
+				(font
+					(size 1.27 1.27)
+				)
+				(justify bottom)
+				(hide yes)
+			)
+		)
+		(property "Manufacturer Part No" "1070TR"
+			(at 91.44 82.55 90)
+			(effects
+				(font
+					(size 1.27 1.27)
+				)
+				(hide yes)
+			)
+		)
+		(pin "N"
+		)
+		(pin "P"
+		)
+		(instances
+			(project ""
+				(path "/8e21fa9a-50eb-4ff7-ab75-73c4d6c5f942/83536851-927e-4d27-972f-18188fbc94fe"
+					(reference "BT1")
+					(unit 1)
+				)
+			)
+		)
+	)
+	(symbol
 		(lib_id "Timer:ICM7555xB")
 		(at 200.66 120.65 0)
@@
 	)
 	(symbol
-		(lib_id "Connector:Conn_01x02_Pin")
-		(at 99.06 74.93 0)
-		(mirror y)
-		(unit 1)
-		(exclude_from_sim no)
-		(in_bom yes)
-		(on_board yes)
-		(dnp no)
-		(property "Reference" "J1"
-			(at 98.425 69.85 0)
-			(effects
-				(font
-					(size 1.27 1.27)
-				)
-			)
-		)
-		(property "Value" "BatteryHolder"
-			(at 99.06 72.644 0)
-			(effects
-				(font
-					(size 1.27 1.27)
-				)
-			)
-		)
-		(property "Footprint" "Battery:BatteryHolder_Keystone_1060_1x2032"
-			(at 99.06 74.93 0)
-			(effects
-				(font
-					(size 1.27 1.27)
-				)
-				(hide yes)
-			)
-		)
-		(property "Datasheet" "~"
-			(at 99.06 74.93 0)
-			(effects
-				(font
-					(size 1.27 1.27)
-				)
-				(hide yes)
-			)
-		)
-		(property "Description" "Battery Holder (Open) Coin, 20.0mm 1 Cell SMD (SMT) Tab"
-			(at 99.06 74.93 0)
-			(effects
-				(font
-					(size 1.27 1.27)
-				)
-				(hide yes)
-			)
-		)
-		(property "Manufacturer Part No" "1057TR"
-			(at 99.06 74.93 0)
-			(effects
-				(font
-					(size 1.27 1.27)
-				)
-				(hide yes)
-			)
-		)
-		(pin "2"
-		)
-		(pin "1"
-		)
-		(instances
-			(project "PinCheck-4"
-				(path "/8e21fa9a-50eb-4ff7-ab75-73c4d6c5f942/83536851-927e-4d27-972f-18188fbc94fe"
-					(reference "J1")
-					(unit 1)
-				)
-			)
-		)
-	)
-	(symbol
 		(lib_id "Device:R")
 		(at 241.3 109.22 0)
@@
 	(symbol
 		(lib_id "power:PWR_FLAG")
-		(at 82.55 72.39 0)
+		(at 91.44 71.12 0)
 		(unit 1)
 		(exclude_from_sim no)
@@
 		(fields_autoplaced yes)
 		(property "Reference" "#FLG02"
-			(at 82.55 70.485 0)
+			(at 91.44 69.215 0)
 			(effects
 				(font
@@
 		)
 		(property "Value" "PWR_FLAG"
-			(at 82.55 67.31 0)
+			(at 91.44 66.04 0)
 			(effects
 				(font
@@
 		)
 		(property "Footprint" ""
-			(at 82.55 72.39 0)
+			(at 91.44 71.12 0)
 			(effects
 				(font
@@
 		)
 		(property "Datasheet" "~"
-			(at 82.55 72.39 0)
+			(at 91.44 71.12 0)
 			(effects
 				(font
@@
 		)
 		(property "Description" "Special symbol for telling ERC where power comes from"
-			(at 82.55 72.39 0)
+			(at 91.44 71.12 0)
 			(effects
 				(font
@@
 	(symbol
 		(lib_id "power:GND")
-		(at 91.44 83.82 0)
+		(at 91.44 91.44 0)
 		(unit 1)
 		(exclude_from_sim no)
@@
 		(fields_autoplaced yes)
 		(property "Reference" "#PWR020"
-			(at 91.44 90.17 0)
+			(at 91.44 97.79 0)
 			(effects
 				(font
@@
 		)
 		(property "Value" "GND"
-			(at 91.44 88.9 0)
+			(at 91.44 96.52 0)
 			(effects
 				(font
@@
 		)
 		(property "Footprint" ""
-			(at 91.44 83.82 0)
+			(at 91.44 91.44 0)
 			(effects
 				(font
@@
 		)
 		(property "Datasheet" ""
-			(at 91.44 83.82 0)
+			(at 91.44 91.44 0)
 			(effects
 				(font
@@
 		)
 		(property "Description" "Power symbol creates a global label with name \"GND\" , ground"
-			(at 91.44 83.82 0)
-			(effects
-				(font
+			(at 91.44 91.44 0)
+			(effects
+				(font
