File: PinCheck-4/seq_logic.kicad_sch (KiCad schematic)
At the start: 13 parts, among them J2 LEMHAL Header, U3 74HC14, U4 74HC14

Commit message: Daily sync 2025-08-27 16:57
Parts:
- removed D6, D7, D8, D9: 1N5908, Diode_THT:D_DO-201AE_P15.24mm_Horizontal, symbol Diode:1N5908
- added U7: USBLC6-4SC6, Package_TO_SOT_SMD:SOT-23-6, symbol Power_Protection:USBLC6-4SC6
- C11: renamed from C3; footprint (none) -> Capacitor_SMD:C_0805_2012Metric
- C12: renamed from C8; footprint (none) -> Capacitor_SMD:C_0805_2012Metric
- J3: renamed from J2; footprint (none) -> Connector_Molex:SHDRRA4W70P0X254_1X4_1016X1170X580P
- R16: renamed from R14; footprint (none) -> Resistor_SMD:R_0805_2012Metric
- R17: renamed from R13; footprint (none) -> Resistor_SMD:R_0805_2012Metric
- R18: renamed from R12; footprint (none) -> Resistor_SMD:R_0805_2012Metric
- R19: renamed from R11; footprint (none) -> Resistor_SMD:R_0805_2012Metric
- U5: renamed from U3; footprint (none) -> Package_SO:SOIC-14_3.9x8.7mm_P1.27mm
- U6: renamed from U4; footprint (none) -> Package_SO:SOIC-14_3.9x8.7mm_P1.27mm
Connections:
- net GND: now also U7.2 (GND)
- net at J3.4 (Pin_4), R19.1, U5.9: now also U7.6 (I/O4)
- net at J3.3 (Pin_3), R18.1, U5.5: now also U7.4 (I/O3)
- net at J3.1 (Pin_1), R16.1, U5.1: now also U7.1 (I/O1)
- net at J3.2 (Pin_2), R17.1, U5.3: now also U7.3 (I/O2)
- no-connect marks 0 -> 1
Other:
- moved on the sheet: C11, C12, J3, U5G, U6A, U6B, U6C, U6D, U6G

Commit message: Daily sync 2025-08-28 16:55
Other:
- moved on the sheet: J3, R16, R17, R18, R19, U5A, U5B, U5C, U5D, U5E, U5F, U6A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

Commit message: Daily sync 2025-08-29 22:48
Parts:
- C11, C12: Manufacturer Part No (none) -> 0805B104K160CT
- J3: Manufacturer Part No (none) -> 26-60-5040
- R16, R17, R18, R19: Manufacturer Part No (none) -> ERJP6WF1003V
- U5, U6: Manufacturer Part No (none) -> 74HC14D
- U7: Manufacturer Part No (none) -> USBLC6-4SC6

Commit message: Daily sync 2025-08-30 13:49
Parts:
- renumbered U5 to U6, U6 to U7, U7 to U8
Changed lines of the file:
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@@
 		(dnp no)
 		(fields_autoplaced yes)
-		(property "Reference" "U6"
+		(property "Reference" "U7"
 			(at 177.8 58.42 0)
 			(effects
@@
 			(project "PinCheck-4"
 				(path "/8e21fa9a-50eb-4ff7-ab75-73c4d6c5f942/dc8a47c7-af7d-496f-bdd4-71159f816556"
-					(reference "U6")
+					(reference "U7")
 					(unit 1)
 				)
@@
 		(dnp no)
 		(fields_autoplaced yes)
-		(property "Reference" "#PWR040"
+		(property "Reference" "#PWR044"
 			(at 93.98 114.3 0)
 			(effects
@@
 			(project "PinCheck-4"
 				(path "/8e21fa9a-50eb-4ff7-ab75-73c4d6c5f942/dc8a47c7-af7d-496f-bdd4-71159f816556"
-					(reference "#PWR040")
+					(reference "#PWR044")
 					(unit 1)
 				)
@@
 		(dnp no)
 		(fields_autoplaced yes)
-		(property "Reference" "#PWR038"
+		(property "Reference" "#PWR042"
 			(at 71.12 137.16 0)
 			(effects
@@
 			(project "PinCheck-4"
 				(path "/8e21fa9a-50eb-4ff7-ab75-73c4d6c5f942/dc8a47c7-af7d-496f-bdd4-71159f816556"
-					(reference "#PWR038")
+					(reference "#PWR042")
 					(unit 1)
 				)
@@
 		(dnp no)
 		(fields_autoplaced yes)
-		(property "Reference" "U5"
+		(property "Reference" "U6"
 			(at 208.28 58.42 0)
 			(effects
@@
 			(project "PinCheck-4"
 				(path "/8e21fa9a-50eb-4ff7-ab75-73c4d6c5f942/dc8a47c7-af7d-496f-bdd4-71159f816556"
-					(reference "U5")
+					(reference "U6")
 					(unit 5)
 				)
@@
 		(dnp no)
 		(fields_autoplaced yes)
-		(property "Reference" "U6"
+		(property "Reference" "U7"
 			(at 208.28 100.33 0)
 			(effects
@@
 			(project "PinCheck-4"
 				(path "/8e21fa9a-50eb-4ff7-ab75-73c4d6c5f942/dc8a47c7-af7d-496f-bdd4-71159f816556"
-					(reference "U6")
+					(reference "U7")
 					(unit 6)
 				)
@@
 		(dnp no)
 		(fields_autoplaced yes)
-		(property "Reference" "U6"
+		(property "Reference" "U7"
 			(at 177.8 86.36 0)
 			(effects
@@
 			(project "PinCheck-4"
 				(path "/8e21fa9a-50eb-4ff7-ab75-73c4d6c5f942/dc8a47c7-af7d-496f-bdd4-71159f816556"
-					(reference "U6")
+					(reference "U7")
 					(unit 3)
 				)
@@
 		(dnp no)
 		(fields_autoplaced yes)
-		(property "Reference" "U6"
+		(property "Reference" "U7"
 			(at 177.8 72.39 0)
 			(effects
@@
 			(project "PinCheck-4"
 				(path "/8e21fa9a-50eb-4ff7-ab75-73c4d6c5f942/dc8a47c7-af7d-496f-bdd4-71159f816556"
-					(reference "U6")
+					(reference "U7")
 					(unit 2)
 				)
@@
 		(dnp no)
 		(fields_autoplaced yes)
-		(property "Reference" "#PWR034"
+		(property "Reference" "#PWR038"
 			(at 25.4 156.21 0)
 			(effects
@@
 			(project "PinCheck-4"
 				(path "/8e21fa9a-50eb-4ff7-ab75-73c4d6c5f942/dc8a47c7-af7d-496f-bdd4-71159f816556"
-					(reference "#PWR034")
+					(reference "#PWR038")
 					(unit 1)
 				)
@@
 		(dnp no)
 		(fields_autoplaced yes)
-		(property "Reference" "U5"
+		(property "Reference" "U6"
 			(at 158.75 86.36 0)
 			(effects
@@
 			(project "PinCheck-4"
 				(path "/8e21fa9a-50eb-4ff7-ab75-73c4d6c5f942/dc8a47c7-af7d-496f-bdd4-71159f816556"
-					(reference "U5")
+					(reference "U6")
 					(unit 3)
 				)
@@
 		(dnp no)
 		(fields_autoplaced yes)
-		(property "Reference" "U6"
+		(property "Reference" "U7"
 			(at 177.8 100.33 0)
 			(effects
@@
 			(project "PinCheck-4"
 				(path "/8e21fa9a-50eb-4ff7-ab75-73c4d6c5f942/dc8a47c7-af7d-496f-bdd4-71159f816556"
-					(reference "U6")
+					(reference "U7")
 					(unit 4)
 				)
@@
 		(dnp no)
 		(fields_autoplaced yes)
-		(property "Reference" "U6"
+		(property "Reference" "U7"
 			(at 208.28 86.36 0)
 			(effects
@@
 			(project "PinCheck-4"
 				(path "/8e21fa9a-50eb-4ff7-ab75-73c4d6c5f942/dc8a47c7-af7d-496f-bdd4-71159f816556"
-					(reference "U6")
+					(reference "U7")
 					(unit 5)
 				)
@@
 		(on_board yes)
 		(dnp no)
-		(property "Reference" "U5"
+		(property "Reference" "U6"
 			(at 158.75 100.33 0)
 			(effects
@@
 			(project "PinCheck-4"
 				(path "/8e21fa9a-50eb-4ff7-ab75-73c4d6c5f942/dc8a47c7-af7d-496f-bdd4-71159f816556"
-					(reference "U5")
+					(reference "U6")
 					(unit 4)
 				)
@@
 		(dnp no)
 		(fields_autoplaced yes)
-		(property "Reference" "U7"
+		(property "Reference" "U8"
 			(at 100.33 95.2499 0)
 			(effects
@@
 			(project ""
 				(path "/8e21fa9a-50eb-4ff7-ab75-73c4d6c5f942/dc8a47c7-af7d-496f-bdd4-71159f816556"
-					(reference "U7")
+					(reference "U8")
 					(unit 1)
 				)
@@
 		(dnp no)
 		(fields_autoplaced yes)
-		(property "Reference" "#PWR039"
+		(property "Reference" "#PWR043"
 			(at 71.12 190.5 0)
 			(effects
@@
 			(project "PinCheck-4"
 				(path "/8e21fa9a-50eb-4ff7-ab75-73c4d6c5f942/dc8a47c7-af7d-496f-bdd4-71159f816556"
-					(reference "#PWR039")
+					(reference "#PWR043")
 					(unit 1)
 				)
@@
 		(dnp no)
 		(fields_autoplaced yes)
-		(property "Reference" "#PWR041"
+		(property "Reference" "#PWR045"
 			(at 128.27 123.19 0)
 			(effects
@@
 			(project "PinCheck-4"
 				(path "/8e21fa9a-50eb-4ff7-ab75-73c4d6c5f942/dc8a47c7-af7d-496f-bdd4-71159f816556"
-					(reference "#PWR041")
+					(reference "#PWR045")
 					(unit 1)
 				)
@@
 		(dnp no)
 		(fields_autoplaced yes)
-		(property "Reference" "#PWR037"
+		(property "Reference" "#PWR041"
 			(at 55.88 156.21 0)
 			(effects
@@
 			(project "PinCheck-4"
 				(path "/8e21fa9a-50eb-4ff7-ab75-73c4d6c5f942/dc8a47c7-af7d-496f-bdd4-71159f816556"
-					(reference "#PWR037")
+					(reference "#PWR041")
 					(unit 1)
 				)
@@
 		(dnp no)
 		(fields_autoplaced yes)
-		(property "Reference" "U5"
+		(property "Reference" "U6"
 			(at 158.75 58.42 0)
 			(effects
@@
 			(project "PinCheck-4"
 				(path "/8e21fa9a-50eb-4ff7-ab75-73c4d6c5f942/dc8a47c7-af7d-496f-bdd4-71159f816556"
-					(reference "U5")
+					(reference "U6")
 					(unit 1)
 				)
@@
 		(dnp no)
 		(fields_autoplaced yes)
-		(property "Reference" "U5"
+		(property "Reference" "U6"
 			(at 46.99 167.6399 0)
 			(effects
@@
 			(project "PinCheck-4"
 				(path "/8e21fa9a-50eb-4ff7-ab75-73c4d6c5f942/dc8a47c7-af7d-496f-bdd4-71159f816556"
-					(reference "U5")
+					(reference "U6")
 					(unit 7)
 				)
@@
 		(dnp no)
 		(fields_autoplaced yes)
-		(property "Reference" "U6"
+		(property "Reference" "U7"
 			(at 77.47 167.6399 0)
 			(effects
@@
 			(project "PinCheck-4"
 				(path "/8e21fa9a-50eb-4ff7-ab75-73c4d6c5f942/dc8a47c7-af7d-496f-bdd4-71159f816556"
-					(reference "U6")
+					(reference "U7")
 					(unit 7)
 				)
@@
 		(dnp no)
 		(fields_autoplaced yes)
-		(property "Reference" "#PWR036"
+		(property "Reference" "#PWR040"
 			(at 40.64 190.5 0)
 			(effects
@@
 			(project "PinCheck-4"
 				(path "/8e21fa9a-50eb-4ff7-ab75-73c4d6c5f942/dc8a47c7-af7d-496f-bdd4-71159f816556"
-					(reference "#PWR036")
+					(reference "#PWR040")
 					(unit 1)
 				)
@@
 		(dnp no)
 		(fields_autoplaced yes)
-		(property "Reference" "U5"
+		(property "Reference" "U6"
 			(at 158.75 72.39 0)
 			(effects
@@
 			(project "PinCheck-4"
 				(path "/8e21fa9a-50eb-4ff7-ab75-73c4d6c5f942/dc8a47c7-af7d-496f-bdd4-71159f816556"
-					(reference "U5")
+					(reference "U6")
 					(unit 2)
 				)
@@
 		(dnp no)
 		(fields_autoplaced yes)
-		(property "Reference" "#PWR035"
+		(property "Reference" "#PWR039"
 			(at 40.64 137.16 0)
 			(effects
@@
 			(project "PinCheck-4"
 				(path "/8e21fa9a-50eb-4ff7-ab75-73c4d6c5f942/dc8a47c7-af7d-496f-bdd4-71159f816556"
-					(reference "#PWR035")
+					(reference "#PWR039")
 					(unit 1)
 				)
@@
 		(dnp no)
 		(fields_autoplaced yes)
-		(property "Reference" "U5"
+		(property "Reference" "U6"
 			(at 208.28 72.39 0)
 			(effects
@@
 			(project "PinCheck-4"
 				(path "/8e21fa9a-50eb-4ff7-ab75-73c4d6c5f942/dc8a47c7-af7d-496f-bdd4-71159f816556"
-					(reference "U5")
+					(reference "U6")
 					(unit 6)
 				)

Commit message: Daily sync 2025-09-01 11:59
Parts:
- removed J3: LEMHAL Header, Connector_Molex:SHDRRA4W70P0X254_1X4_1016X1170X580P, symbol Connector:Conn_01x04_Socket
- added J2: LEMHAL Header, Connector:CONN_A-7478-04A_MOL, symbol PinCheck-4_Library:22053041
Connections:
- net at R19.1, U6.9, U8.6 (I/O4): now also J2.4
- net at R18.1, U6.5, U8.4 (I/O3): now also J2.3
- net at R16.1, U6.1, U8.1 (I/O1): now also J2.1
- net at R17.1, U6.3, U8.3 (I/O2): now also J2.2
Changed lines of the file:
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@@
+	)
+	(symbol
+		(lib_id "PinCheck-4_Library:22053041")
+		(at 60.96 67.31 0)
+		(mirror y)
+		(unit 1)
+		(exclude_from_sim no)
+		(in_bom yes)
+		(on_board yes)
+		(dnp no)
+		(fields_autoplaced yes)
+		(property "Reference" "J2"
+			(at 52.07 59.69 0)
+			(effects
+				(font
+					(size 1.524 1.524)
+				)
+			)
+		)
+		(property "Value" "LEMHAL Header"
+			(at 52.07 62.23 0)
+			(effects
+				(font
+					(size 1.524 1.524)
+				)
+			)
+		)
+		(property "Footprint" "Connector:CONN_A-7478-04A_MOL"
+			(at 60.96 67.31 0)
+			(effects
+				(font
+					(size 1.27 1.27)
+					(italic yes)
+				)
+				(hide yes)
+			)
+		)
+		(property "Datasheet" "https://www.molex.com/en-us/products/part-detail-pdf/22053041?display=pdf"
+			(at 60.96 67.31 0)
+			(effects
+				(font
+					(size 1.27 1.27)
+					(italic yes)
+				)
+				(hide yes)
+			)
+		)
+		(property "Description" "Pin Header, Signal, Wire-to-Board, 2.54 mm, 1 Rows, 4 Contacts, Through Hole Right Angle"
+			(at 60.96 67.31 0)
+			(effects
+				(font
+					(size 1.27 1.27)
+				)
+				(hide yes)
+			)
+		)
+		(property "Manufacturer Part No" "22-05-3041"
+			(at 60.96 67.31 0)
+			(effects
+				(font
+					(size 1.27 1.27)
+				)
+				(hide yes)
+			)
+		)
+		(pin "2"
+		)
+		(pin "1"
+		)
+		(pin "4"
+		)
+		(pin "3"
+		)
+		(instances
+			(project ""
+				(path "/8e21fa9a-50eb-4ff7-ab75-73c4d6c5f942/dc8a47c7-af7d-496f-bdd4-71159f816556"
+					(reference "J2")
+					(unit 1)
+				)
+			)
+		)
 	)
 	(symbol
@@
 					(unit 1)
 				)
-			)
-		)
-	)
-	(symbol
-		(lib_id "Connector:Conn_01x04_Socket")
-		(at 55.88 69.85 0)
-		(mirror y)
-		(unit 1)
-		(exclude_from_sim no)
-		(in_bom yes)
-		(on_board yes)
-		(dnp no)
-		(fields_autoplaced yes)
-		(property "Reference" "J3"
-			(at 56.515 62.23 0)
-			(effects
-				(font
-					(size 1.27 1.27)
-				)
-			)
-		)
-		(property "Value" "LEMHAL Header"
-			(at 56.515 64.77 0)
-			(effects
-				(font
-					(size 1.27 1.27)
-				)
-			)
-		)
-		(property "Footprint" "Connector_Molex:SHDRRA4W70P0X254_1X4_1016X1170X580P"
-			(at 55.88 69.85 0)
-			(effects
-				(font
-					(size 1.27 1.27)
-				)
-				(hide yes)
-			)
-		)
-		(property "Datasheet" "~"
-			(at 55.88 69.85 0)
-			(effects
-				(font
-					(size 1.27 1.27)
-				)
-				(hide yes)
-			)
-		)
-		(property "Description" "Pin Header, Right Angle, Power, 3.96 mm, 1 Rows, 4 Contacts, Through Hole Right Angle, KK 396 41792"
-			(at 55.88 69.85 0)
-			(effects
-				(font
-					(size 1.27 1.27)
-				)
-				(hide yes)
-			)
-		)
-		(property "Manufacturer Part No" "26-60-5040"
-			(at 55.88 69.85 0)
-			(effects
-				(font
-					(size 1.27 1.27)
-				)
-				(hide yes)
-			)
-		)
-		(pin "2"
-		)
-		(pin "4"
-		)
-		(pin "1"
-		)
-		(pin "3"
-		)
-		(instances
-			(project "PinCheck-4"
-				(path "/8e21fa9a-50eb-4ff7-ab75-73c4d6c5f942/dc8a47c7-af7d-496f-bdd4-71159f816556"
-					(reference "J3")
-					(unit 1)
-				)
