File: PinCheck-4/spdt_logic.kicad_sch (KiCad schematic)
At the start: 11 parts, among them J2 DA15_Socket, SW2 SW_SPST, U3 4017, U4 TMUX1574DYY

Commit message: Daily sync 2025-08-29 22:48
Parts:
- C10, C9: Manufacturer Part No (none) -> 0805B104K160CT
- J2: footprint Connector_Dsub:DSUB-15_Socket_Horizontal_P2.77x2.54mm_EdgePinOffset9.40mm -> Connector_Dsub:DSUB-15_Socket_Horizontal_P2.77x2.84mm_EdgePinOffset9.90mm_Housed_MountingHolesOffset11.32mm; Manufacturer Part No (none) -> MHDD15-F-T-B-S-R
- R11, R12, R13, R14: Manufacturer Part No (none) -> MCMR08X1001FTL
- R15: Manufacturer Part No (none) -> ERJP6WF1003V
- SW2: Manufacturer Part No (none) -> Dip Switch SPST 1 Position Through Hole Slide (Standard) Ac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
- U3: Manufacturer Part No (none) -> CD4017BM96
- U4: Manufacturer Part No (none) -> 4 Circuit IC Switch 2:1 4.5Ohm 16-SOT-23-THIN
Changed lines of the file:
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@@
 			)
 		)
-		(property "Description" "Resistor"
+		(property "Description" "SMD Chip Resistor, 100 kohm, ± 1%, 500 mW, 0805 [2012 Metric], Thick Film (Double Sided)"
+			(at 168.91 127 0)
+			(effects
+				(font
+					(size 1.27 1.27)
+				)
+				(hide yes)
+			)
+		)
+		(property "Manufacturer Part No" "ERJP6WF1003V"
 			(at 168.91 127 0)
 			(effects
@@
 			)
 		)
-		(property "Description" "Low Capacitance, 4-Channel, 2 to 1 Switch, Powered-off Protection with 1.8V logic, TSOT-23-16"
+		(property "Description" "4 Circuit IC Switch 2:1 4.5Ohm 16-SOT-23-THIN"
 			(at 194.31 71.12 0)
+			(effects
+				(font
+					(size 1.27 1.27)
+				)
+				(hide yes)
+			)
+		)
+		(property "Manufacturer Part No" "4 Circuit IC Switch 2:1 4.5Ohm 16-SOT-23-THIN"
+			(at 194.31 106.68 0)
 			(effects
 				(font
@@
 			)
 		)
-		(property "Description" "Resistor"
+		(property "Description" "SMD Chip Resistor, Ceramic, 1 kohm, ± 1%, 125 mW, 0805 [2012 Metric], Thick Film, Sulfur Resistant"
 			(at 127 99.06 0)
+			(effects
+				(font
+					(size 1.27 1.27)
+				)
+				(hide yes)
+			)
+		)
+		(property "Manufacturer Part No" "MCMR08X1001FTL"
+			(at 127 99.06 90)
 			(effects
 				(font
@@
 			)
 		)
-		(property "Description" "Resistor"
+		(property "Description" "SMD Chip Resistor, Ceramic, 1 kohm, ± 1%, 125 mW, 0805 [2012 Metric], Thick Film, Sulfur Resistant"
 			(at 133.35 101.6 0)
+			(effects
+				(font
+					(size 1.27 1.27)
+				)
+				(hide yes)
+			)
+		)
+		(property "Manufacturer Part No" "MCMR08X1001FTL"
+			(at 133.35 101.6 90)
 			(effects
 				(font
@@
 			)
 		)
-		(property "Description" "Single Pole Single Throw (SPST) switch"
+		(property "Description" "Dip Switch SPST 1 Position Through Hole Slide (Standard) Actuator 25mA 24VDC"
+			(at 158.75 121.92 0)
+			(effects
+				(font
+					(size 1.27 1.27)
+				)
+				(hide yes)
+			)
+		)
+		(property "Manufacturer Part No" "Dip Switch SPST 1 Position Through Hole Slide (Standard) Actuator 25mA 24VDC"
 			(at 158.75 121.92 0)
 			(effects
@@
 			)
 		)
-		(property "Description" "Unpolarized capacitor"
+		(property "Description" "SMD Multilayer Ceramic Capacitor, 0.1 µF, 16 V, 0805 [2012 Metric], ± 10%, X7R"
+			(at 179.07 73.66 0)
+			(effects
+				(font
+					(size 1.27 1.27)
+				)
+				(hide yes)
+			)
+		)
+		(property "Manufacturer Part No" "0805B104K160CT"
 			(at 179.07 73.66 0)
 			(effects
@@
 			)
 		)
-		(property "Description" "Resistor"
+		(property "Description" "SMD Chip Resistor, Ceramic, 1 kohm, ± 1%, 125 mW, 0805 [2012 Metric], Thick Film, Sulfur Resistant"
 			(at 114.3 93.98 0)
+			(effects
+				(font
+					(size 1.27 1.27)
+				)
+				(hide yes)
+			)
+		)
+		(property "Manufacturer Part No" "MCMR08X1001FTL"
+			(at 114.3 93.98 90)
 			(effects
 				(font
@@
 			)
 		)
-		(property "Footprint" "Connector_Dsub:DSUB-15_Socket_Horizontal_P2.77x2.54mm_EdgePinOffset9.40mm"
+		(property "Footprint" "Connector_Dsub:DSUB-15_Socket_Horizontal_P2.77x2.84mm_EdgePinOffset9.90mm_Housed_MountingHolesOffset11.32mm"
 			(at 241.3 104.14 0)
 			(effects
@@
 			)
 		)
-		(property "Description" "15-pin D-SUB connector, socket (female) (low-density/2 columns)"
+		(property "Description" "MH Connectors MHDD 15 Way Right Angle Through Hole D-sub Connector Socket, 2.77mm Pitch"
+			(at 241.3 104.14 0)
+			(effects
+				(font
+					(size 1.27 1.27)
+				)
+				(hide yes)
+			)
+		)
+		(property "Manufacturer Part No" "MHDD15-F-T-B-S-R "
 			(at 241.3 104.14 0)
 			(effects
@@
 			)
 		)
-		(property "Description" "Resistor"
+		(property "Description" "SMD Chip Resistor, Ceramic, 1 kohm, ± 1%, 125 mW, 0805 [2012 Metric], Thick Film, Sulfur Resistant"
 			(at 120.65 96.52 0)
+			(effects
+				(font
+					(size 1.27 1.27)
+				)
+				(hide yes)
+			)
+		)
+		(property "Manufacturer Part No" "MCMR08X1001FTL"
+			(at 120.65 96.52 90)
 			(effects
 				(font
@@
 			)
 		)
-		(property "Description" "Unpolarized capacitor"
+		(property "Description" "SMD Multilayer Ceramic Capacitor, 0.1 µF, 16 V, 0805 [2012 Metric], ± 10%, X7R"
+			(at 67.31 76.2 0)
+			(effects
+				(font
+					(size 1.27 1.27)
+				)
+				(hide yes)
+			)
+		)
+		(property "Manufacturer Part No" "0805B104K160CT"
 			(at 67.31 76.2 0)
 			(effects
@@
 			)
 		)
-		(property "Description" "Johnson Counter ( 10 outputs )"
+		(property "Description" "Counter IC Counter, Decade 1 Element 10 Bit Positive, Negative 16-SOIC"
 			(at 82.55 106.68 0)
 			(effects
+				(font
+					(size 1.27 1.27)
+				)
+				(hide yes)
+			)
+		)
+		(property "Manufacturer Part No" "CD4017BM96"
+			(at 82.55 106.68 0)
+			(effects

Commit message: Daily sync 2025-08-30 13:49
Parts:
- removed SW2: SW_SPST, Button_Switch_THT:SW_DIP_SPSTx01_Slide_9.78x4.72mm_W7.62mm_P2.54mm, symbol Switch:SW_SPST
- added SW2: OS102011MA1QS1, Button_Switch_THT:OS102011MA1QS1, symbol Switch:OS102011MA1QS1
- renumbered U3 to U4, U4 to U5
Connections:
- net GND: now also SW2.MH1, SW2.MH2
- net VCC: now also SW2.1 (NO)
- net at R15.1, U5.1 (SEL): now also SW2.2 (COM)
Other:
- moved on the sheet: R15

Commit message: Daily sync 2025-09-01 11:59
Parts:
- renumbered J2 to J1
Changed lines of the file:
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@@
 		(dnp no)
 		(fields_autoplaced yes)
-		(property "Reference" "J2"
+		(property "Reference" "J1"
 			(at 246.38 102.8699 0)
 			(effects
@@
 			(project "PinCheck-4"
 				(path "/8e21fa9a-50eb-4ff7-ab75-73c4d6c5f942/9f925a3b-1ca7-46c5-bc3a-22e483273a15"
-					(reference "J2")
+					(reference "J1")
 					(unit 1)
 				)
